File: fz10_pow.brd (EAGLE design)
At the start: 107 x 100 mm, 71 parts, among them T1 TRANS_ER29

Commit message: .
Parts:
- removed C1: 47x400v, rcl:EB22,5D
- removed C10: 10n*, rcl:C050-025X075
- removed C100: 220nx250v, 3do:C_26X19
- removed C101: (no value), rcl:E5-10,5
- removed C102: 100mfx25v, rcl:E5-13
- removed C103: 470mfx25v, rcl:E5-8,5
- removed C11: 4n7, rcl:C050-025X075
- removed C12A, C12B, C2, C4, C5, C7: (no value), rcl:C050-025X075
- removed C12C, C12D: (no value), rcl:C1206
- removed C3: 100x25v, rcl:E2,5-6
- removed C6: 100n, rcl:C1206
- removed C8: (no value), rcl:E5-8,5
- removed D1, D2, D3, D4: 1N4004, diode:DO41-10
- removed D5: (no value), diode:DO34Z7
- removed D6, D7: BYV32, diode:TO220ABS
- removed DA1: UC3842N, v-reg:DIL08
- removed F1: (no value), fuse:SHK20L
- removed L1: LFLF-10X13, DSS0:LF-10X13
- removed L2, L3: (no value), rcl:TFI0305
- removed R1, R10, R11, R11A, R11B, R17B, R2, R4, R5, R6, R7, R8, R9: (no value), rcl:R1206
- removed R1-2, R3: (no value), rcl:P0613/15
- removed R12: 910, rcl:R1206
- removed R13: 820, rcl:R1206
- removed R14: 47k*, rcl:R1206
- removed R155A: 82k, rcl:M1206
- removed R155B, R155C: (no value), rcl:M1206
- removed R156: 3k9, rcl:M1206
- removed R16: 3k3, rcl:R1206
- removed R17: (no value), rcl:RTRIM3296W
- removed R20: 100, rcl:P0613/15
- removed T1: TRANS_ER29, 3do:ER29
- removed VD1: 1N4148DO35-10, diode:DO35-10
- removed VD2, VD3, VD6, VD7: 1N4148DO35-7, diode:DO35-7
- removed VT1: IRF3704L-V, transistor-power:TO262-V
- added 1C1: 220nX250v, 3do:C_26X19
- added 1C2: 100nX250v, rcl:C150-084X183
- added 1C7: 47x400v, rcl:EB22,5D
- added 1DA1: UC3842N, v-reg:DIL08
- added 1F1: (no value), fuse:SHK20L
- added 1L1: LFLF-10X13, DSS0:LF-10X13
- added 1R1: 470k, rcl:P0613/15
- added 1RZ1: (no value), varistor:S1210
- added 1TH1: (no value), varistor:R-7,5
- added 1VD1, 1VD2, 1VD3, 1VD4: 1N4007, diode:DO41-10
- added 1VD1B: S1WBS60, rectifier:B-DIL
- added 2C10: 10n*, rcl:C050-025X075
- added 2C11: 4n7, rcl:C050-025X075
- added 2C2: 10n, rcl:C050-025X075
- added 2C3: 100x25v, rcl:E2,5-6
- added 2C4, 2C5, 2C7, 4C2A, 4C2B: (no value), rcl:C050-025X075
- added 2C6: 100n, rcl:C1206
- added 2R1: 220k 1w, rcl:P0613/15
- added 2R10: 1k, rcl:R1206
- added 2R11A, 2R11B, 2R11C, 2R11D: 1, rcl:R0805
- added 2R12: 910, rcl:R1206
- added 2R13: 820, rcl:R1206
- added 2R14: 47k*, rcl:R1206
- added 2R16: 3k3, rcl:R1206
- added 2R3: 80k 1w, rcl:P0613/15
- added 2R4: 22, rcl:R1206
- added 2R5, 2R7, 2R8, 2R9, 4R1B: (no value), rcl:R1206
- added 2T1: TRANS_ER29, 3do:ER29
- added 2VD1: 1N4148DO35-10, diode:DO35-10
- added 2VD2, 2VD3, 4VD3: 1N4148DO35-7, diode:DO35-7
- added 2VD4: (no value), diode:DO34Z7
- added 2VT1: IRF3704L-V, transistor-power:TO262-V
- added 3C1: (no value), rcl:E5-10,5
- added 3C2: 100mfx25v, rcl:E5-13
- added 3C3: 470mfx25v, rcl:E5-8,5
- added 3C5: (no value), rcl:E5-8,5
- added 3L1, 3L2: (no value), rcl:TFI0305
- added 3R5A: 82k, rcl:M1206
- added 3R5B, 3R5C: (no value), rcl:M1206
- added 3R6: 3k9, rcl:M1206
- added 3R7: 100, rcl:P0613/15
- added 3VD1, 3VD2: BYV32, diode:TO220ABS
- added 4C2C, 4C2D: (no value), rcl:C1206
- added 4C3: 4m7, rcl:E2,5-5
- added 4R1C: (no value), rcl:RTRIM3296W
- added 4R2, 4R3: 4k7, rcl:R1206
- added 4VD1: LL4148, diode:SOD80C
- added 4VD2: LL4158, diode:SOD80C
- added J5V, J9V, JGND, JMON: (no value), pinhead:1X01
- 4R4: value (none) -> 2k
- 4R5: value (none) -> 1k
- 4VT1: value (none) -> KT315
- moved DA2 28.8 mm to (81.3, 12.7), turned to 180 degrees
- moved OK1 2.84 mm to (72.4, 25.4)
- renumbered C14 to 4C1, DD1 to 4DD1, R17A to 4R1A, R18 to 4R4, R19 to 4R5, T2 to 4VT1
Connections:
- removed net N$38: R2.2, R6.2
- new net N$29: 1C2.2, 1L1.2, 1VD1B.AC1, 1VD2.A, 1VD4.C
- new net N$37: 2R11A.1, 2R11B.1, 2R11C.2, 2R11D.2
- net +5V: now also 3C3.+, 3L2.2, 3R6.2, 4C3.+, J5V.1; no longer C103.+, L3.2, R156.2
- net +9V: now also 3C5.+, 3L1.2, 3R5A.2, 3R7.2, J9V.1; no longer C8.+, L2.2, R155A.2, R20.2
- net -IN: now also 1C7.-, 1DA1.5, 1VD1B.-, 1VD3.A, 1VD4.A, 2C11.1, 2C3.-, 2C5.2, 2C6.2, 2C7.2, 2R10.2, 2R11C.1, 2R11D.1, 2R7.1, 2T1.2, 2VD4.A; no longer C1.-, C11.1, C3.-, C5.2, C6.2, C7.2, D3.A, D4.A, D5.A, DA1.5, R10.2, R11A.1, R11B.1, R7.1, T1.2
- net GND: now also 2C11.2, 2R16.1, 2T1.11, 2T1.7, 3C1.-, 3C2.-, 3C3.-, 3C5.-, 3R7.1, 4R3.1, 4VD3.A, JGND.1; no longer C101.-, C102.-, C103.-, C11.2, C8.-, R16.1, R20.1, T1.11, T1.7
- net MON: now also JMON.1
- net N$1: now also 4C2A.2, 4C2B.2, 4C2C.2, 4C2D.2, 4R1C.3, 4VD1.A; no longer C12A.2, C12B.2, C12C.2, C12D.2, R17.3, VD6.A
- net N$10: now also 4R1B.1, 4R1C.2, 4VD1.C, 4VD2.C; no longer R17.2, R17B.1, VD6.C, VD7.C
- net N$11: now also 2R9.2, 2VD3.A, 2VT1.1; no longer R9.2, VD3.A, VT1.1
- net N$12: now also 2R12.1, 2R13.2; no longer R12.1, R13.2
- net N$13: now also 2R12.2, 3C2.+, 3L2.1, 3VD2.C; no longer C102.+, D7.C, L3.1, R12.2
- net N$14: now also 2R13.1, 2R14.1; no longer R13.1, R14.1
- net N$15: now also 1C2.1, 1L1.4, 1VD1.A, 1VD1B.AC2, 1VD3.C; no longer D1.A, D3.C, L1.4
- net N$16: now also 2C10.2, 2R14.2; no longer C10.2, R14.2
- net N$17: now also 2T1.4, 2VD2.A, 2VT1.2; no longer T1.5, VD2.A, VT1.2
- net N$18: now also 1F1.1A; no longer F1.1A
- net N$19: now also 4C2A.1, 4C2B.1, 4C2C.1, 4C2D.1, 4R1B.2, 4R1C.1, 4VD2.A; no longer C12A.1, C12B.1, C12C.1, C12D.1, R17.1, R17B.2, VD7.A
- net N$20: now also 1DA1.8, 2C6.1, 2R8.2; no longer C6.1, DA1.8, R8.2
- net N$21: now also 2R11A.2, 2R11B.2, 2VT1.3; no longer R11A.2, R11B.2, VT1.3
- net N$22: now also 2R4.2, 2VD1.C; no longer R4.2, VD1.C
- net N$23: now also 1C7.+, 1VD1.C, 1VD1B.+, 1VD2.C, 2C2.1, 2R1.2, 2R3.2, 2T1.5; no longer C1.+, C2.1, D1.C, D2.C, R1-2.2, R3.2, T1.4
- net N$24: now also 2T1.1, 2VD1.A; no longer T1.1, VD1.A
- net N$27: now also 3R5A.1, 3R5B.2; no longer R155A.1, R155B.2
- net N$28: now also 2T1.10, 3VD2.A1, 3VD2.A2; no longer D7.A1, D7.A2, T1.10
- net N$3: now also 1DA1.4, 2C5.1, 2R8.1; no longer C5.1, DA1.4, R8.1
- net N$30: now also 2C2.2, 2R3.1, 2VD2.C; no longer C2.2, R3.1, VD2.C
- net N$31: now also 4DD1.8, 4R2.1, 4R3.2; no longer R1.2, R2.1
- net N$32: now also 1C1.2, 1L1.1, 1R1.1, 1RZ1.2, PCB.SW1; no longer C100.2, L1.3, PCB.SW2, R11.1
- net N$33: now also 1C1.1, 1L1.3, 1R1.2, 1RZ1.1, 1TH1.2; no longer C100.1, F1.2A, L1.1, R1.1
- net N$34: now also PCB.SW2; no longer PCB.SW1
- net N$35: now also 4C3.-, 4R2.2, 4VD3.C; no longer R11.2, R6.1
- net N$36: now also 1F1.2A, 1TH1.1; no longer D2.A, D4.C, L1.2
- net N$39: now also 3C1.+, 3L1.1, 3VD1.C; no longer C101.+, D6.C, L2.1
- net N$4: now also 1DA1.3, 2C7.1, 2R10.1; no longer C7.1, DA1.3, R10.1
- net N$40: now also 1DA1.2, 2C4.2, 2R5.1, 2R7.2; no longer C4.2, DA1.2, R5.1, R7.2
- net N$41: now also 3R5B.1, 3R5C.2; no longer R155B.1, R155C.2
- net N$42: now also 2C10.1, 2R16.2, 3R5C.1, 3R6.1; no longer C10.1, R155C.1, R156.1, R16.2
- net N$5: now also 2T1.6, 3VD1.A1, 3VD1.A2; no longer D6.A1, D6.A2, T1.6
- net N$6: now also 1DA1.1, 2C4.1, 2R5.2; no longer C4.1, DA1.1, R5.2
- net N$7: no longer 4DD1.8
- net N$8: now also 1DA1.6, 2R9.1, 2VD3.C; no longer DA1.6, R9.1, VD3.C
- net N$9: now also 1DA1.7, 2C3.+, 2R1.1, 2R4.1, 2VD4.C; no longer C3.+, D5.C, DA1.7, R1-2.1, R4.1
Routing:
- net -IN: track 30.9 -> 155.6 mm, vias 0 -> 2
- net GND: track 29.1 -> 94.1 mm
- net N$23: track 45.1 -> 102.8 mm, vias 2 -> 0
- net N$32: track 26.9 -> 79.3 mm
- net N$34: track 0.00 -> 45.3 mm
- net N$15: track 0.00 -> 38.0 mm
- net N$33: track 0.00 -> 28.1 mm
- net N$29: track 0.00 -> 22.5 mm
- net N$13: track 0.00 -> 20.5 mm
- net N$39: track 0.00 -> 18.3 mm
- net N$9: track 0.00 -> 18.2 mm
- net N$3: track 0.00 -> 15.3 mm
- net N$40: track 0.00 -> 14.2 mm
- net N$8: track 0.00 -> 12.9 mm
- net N$30: track 0.00 -> 12.2 mm
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Other:
- board text added: "REV1.0"
- board text added: "for FZ-10"

Commit message: .
Parts:
- removed OK1: PC817, optocoupler:DIL04
- added 1PC1: PC817, optocoupler:DIL04
- added 3CN1: (no value), 3do:FTOP-18
- added 3VD3: 12v, diode:DO34Z7
- added 4R6: 100, rcl:M0805
- 1R1: device rcl:P0613/15 -> rcl:0309/12
- 2C4, 2C5, 2C7: value (none) -> 330
- 2C6: device rcl:C1206 -> rcl:C0805
- 2R5: value (none) -> 10k; device rcl:R1206 -> rcl:M0805
- 2R7: value (none) -> 10k
- 2R8: value (none) -> 68k *80ruw
- 2R9: value (none) -> 100
- 2VD1: value 1N4148DO35-10 -> 1N4148
- 2VD2: value 1N4148DO35-7 -> FR207; device diode:DO35-7 -> diode:DO35-10
- 2VD3: value 1N4148DO35-7 -> LL4148; device diode:DO35-7 -> diode:SOD80C
- 3C1: value (none) -> 560mfx25v
- 3C2: value 100mfx25v -> 1000mfx25v
- 3C5: value (none) -> 470vfx25v
- 4VD3: value 1N4148DO35-7 -> (none); device diode:DO35-7 -> diode:SOD80C
- moved 3L2 50.9 mm to (91.4, 57.8)
- moved 3C3 47.0 mm to (91.4, 64.8), turned to 180 degrees
- moved 3C2 44.6 mm to (88.3, 50.2), turned to 180 degrees
- moved 3C1 35.3 mm to (97.2, 30.5), turned to 180 degrees
- moved 3L1 27.3 mm to (105.4, 38.1), turned to 90 degrees
- moved 3R6 23.7 mm to (89.5, 40.0), turned to 90 degrees
- moved 3VD2 18.5 mm to (56.5, 22.2), turned to 90 degrees
- moved 4R1B 16.9 mm to (104.8, 85.1), turned to 270 degrees
- moved 4R1A 16.8 mm to (104.8, 90.8), turned to 270 degrees
- moved 4C3 16.1 mm to (90.2, 71.1), turned to 0 degrees
- moved 1VD3 15.2 mm to (47.0, 59.7)
- moved 4VD3 14.2 mm to (96.5, 71.1), turned to 180 degrees
- moved 3R5C 14.0 mm to (94.6, 38.1)
- moved J5V 13.5 mm to (98.4, 59.7)
- moved 4VD1 13.4 mm to (102.2, 90.8), turned to 90 degrees
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Connections:
- removed net +9V: 3C5.+, 3L1.2, 3R5A.2, 3R7.2, J9V.1
- new net N$38: 3C5.+, 3CN1.1, 3CN1.2, 3CN1.3, 3L1.2, 3R5A.2, 3R7.2, 3VD3.C, J9V.1
- new net N$44: 1C2.1, 1L1.4, 1VD1B.AC1, 1VD2.A, 1VD4.C
- net +5V: now also 3CN1.13, 3CN1.14, 3CN1.15, 3CN1.16, 3CN1.17
- net GND: now also 3CN1.10, 3CN1.11, 3CN1.12, 3CN1.4, 3CN1.5, 3CN1.6, 3CN1.7, 3CN1.8, 3CN1.9, 3VD3.A
- net MON: now also 3CN1.18, 4R6.2; no longer 4R5.1, 4VT1.C
- net N$12: now also 1PC1.2; no longer OK1.2
- net N$13: now also 1PC1.1; no longer OK1.1
- net N$15: now also 1C2.2, 1L1.2; no longer 1C2.1, 1L1.4
- net N$20: now also 1PC1.4; no longer OK1.4
- net N$28: now also 2T1.6; no longer 2T1.10
- net N$29: now also 4R5.1, 4R6.1, 4VT1.C; no longer 1C2.2, 1L1.2, 1VD1B.AC1, 1VD2.A, 1VD4.C
- net N$40: now also 1PC1.3; no longer OK1.3
- net N$5: now also 2T1.10; no longer 2T1.6
Routing:
- net GND: track 94.1 -> 154.9 mm
- net N$44: track 0.00 -> 52.9 mm
- net N$39: track 18.3 -> 68.7 mm
- net N$23: track 102.8 -> 71.0 mm
- net -IN: track 155.6 -> 129.1 mm, vias 2 -> 0
- net N$29: track 22.5 -> 0.00 mm
- net N$5: track 28.1 -> 48.2 mm
- net N$38: track 0.00 -> 17.8 mm
- net +5V: track 0.00 -> 17.8 mm
- net N$28: track 52.8 -> 39.0 mm
- net N$13: track 20.5 -> 10.0 mm
- net N$17: track 39.5 -> 48.3 mm, vias 0 -> 2
- net N$12: track 0.00 -> 6.76 mm
- net N$11: track 10.4 -> 5.33 mm
- net N$15: track 38.0 -> 33.4 mm
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
Commit message: .
Parts:
- 1C1: device 3do:C_26X19 -> 3do:C_26X9
- 2R13: device rcl:R1206 -> rcl:0207/10
- 2R4, 2R9: device rcl:R1206 -> rcl:0204/7
- 2VD1: device diode:DO35-10 -> diode:DO35-7
- 2VD3: device diode:SOD80C -> diode:DO35-7
- 2VD4: device diode:DO34Z7 -> diode:DO35Z10
- 3R5C: device rcl:M1206 -> rcl:0207/10
- 4C2A: value (none) -> 3p
- moved 4R1B 18.0 mm to (92.7, 98.4), turned to 180 degrees
- moved 4VD1 16.1 mm to (87.0, 95.9), turned to 0 degrees
- moved 4R1A 15.5 mm to (89.5, 93.3), turned to 180 degrees
- moved 4VD3 14.8 mm to (109.2, 78.7)
- moved 1VD2 13.7 mm to (34.3, 68.6), turned to 90 degrees
- moved 2C3 13.7 mm to (53.3, 40.0), turned to 180 degrees
- moved 4VD2 13.5 mm to (92.7, 95.2), turned to 180 degrees
- moved 2VD4 12.8 mm to (54.6, 54.0), turned to 0 degrees
- moved 2C2 10.8 mm to (28.6, 54.0), turned to 0 degrees
- moved 4R3 9.44 mm to (89.5, 69.8), turned to 90 degrees
- moved 2R1 9.38 mm to (41.3, 59.1), turned to 180 degrees
- moved 1VD3 9.09 mm to (48.9, 68.6), turned to 270 degrees
- moved 4R1C 8.47 mm to (90.2, 90.8), turned to 90 degrees
- moved 1VD1 8.35 mm to (38.7, 68.6), turned to 90 degrees
- moved 2R16 8.35 mm to (88.3, 21.6)
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Connections:
- net N$15: now also 1C2.1, 1L1.4; no longer 1C2.2, 1L1.2
- net N$19: no longer 4R1B.2, 4R1C.1, 4VD2.A
- net N$44: now also 1C2.2, 1L1.2; no longer 1C2.1, 1L1.4
- net N$7: now also 4R1B.2, 4R1C.1, 4VD2.A
Routing:
- net N$13: track 10.0 -> 66.4 mm
- net GND: track 154.9 -> 196.5 mm
- net -IN: track 129.1 -> 153.8 mm
- net N$15: track 33.4 -> 51.1 mm
- net N$9: track 17.0 -> 34.3 mm
- net N$40: track 11.4 -> 26.4 mm
- net +5V: track 17.8 -> 31.4 mm
- net N$20: track 6.35 -> 16.4 mm
- net N$38: track 17.8 -> 27.3 mm
- net N$14: track 0.00 -> 9.09 mm
- net N$42: track 0.00 -> 7.16 mm
- net N$44: track 52.9 -> 47.7 mm
- net N$27: track 0.00 -> 4.52 mm
- net N$22: track 0.00 -> 4.45 mm
- net N$8: track 12.7 -> 8.25 mm
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
Commit message: .
Parts:
- removed 4C2B: (no value), rcl:C050-025X075
- removed 4C2D: (no value), rcl:C1206
- added 3R6B: 0, rcl:0204/7
- 3R6: device rcl:M1206 -> rcl:0204/7
- 4R6: device rcl:M0805 -> rcl:R1206
- moved 4R1B 20.2 mm to (84.5, 80.0), turned to 270 degrees
- moved 4VD2 18.7 mm to (81.9, 80.0), turned to 270 degrees
- moved 3R6 17.3 mm to (83.8, 52.1), flipped to the top
- moved 3C2 15.3 mm to (79.4, 36.2)
- moved 4C2C 13.9 mm to (84.5, 93.3), turned to 90 degrees
- moved 4R6 13.4 mm to (96.5, 70.2)
- moved 4VD1 11.9 mm to (81.9, 85.1), turned to 90 degrees
- moved 4C2A 11.8 mm to (81.9, 93.3), turned to 90 degrees
- moved 4R4 10.8 mm to (96.5, 76.2)
- moved 1R1 10.3 mm to (61.0, 87.0)
- moved 2C10 10.2 mm to (79.4, 23.5), turned to 180 degrees
- moved 4R1A 9.69 mm to (84.5, 85.1), turned to 270 degrees
- moved 4VT1 9.26 mm to (101.3, 72.1), turned to 90 degrees
- moved 1RZ1 9.09 mm to (64.8, 92.1)
- moved 4R1C 9.09 mm to (88.3, 81.9), turned to 0 degrees
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Connections:
- new net N$43: 3R6.1, 3R6B.2
- net N$1: now also 4DD1.12, 4DD1.13; no longer 4C2B.2, 4C2D.2, 4DD1.1, 4DD1.2
- net N$19: now also 4DD1.1, 4DD1.10, 4DD1.2; no longer 4C2B.1, 4C2D.1, 4DD1.12, 4DD1.13, 4DD1.4
- net N$2: now also 4DD1.11, 4DD1.8, 4DD1.9; no longer 4DD1.3, 4DD1.5, 4DD1.6
- net N$25: now also 4DD1.4; no longer 4DD1.10
- net N$31: now also 4DD1.6; no longer 4DD1.8
- net N$42: now also 3R6B.1; no longer 3R6.1
- net N$7: now also 4DD1.3, 4DD1.5; no longer 4DD1.11, 4DD1.9
Routing:
- net GND: track 196.5 -> 277.0 mm
- net +5V: track 31.4 -> 75.2 mm, vias 0 -> 2
- net N$1: track 0.00 -> 43.5 mm
- net N$2: track 0.00 -> 41.4 mm
- net N$19: track 0.00 -> 28.3 mm
- net N$35: track 0.00 -> 20.7 mm
- net N$31: track 0.00 -> 20.5 mm
- net N$7: track 0.00 -> 19.4 mm
- net N$42: track 7.16 -> 21.8 mm
- net N$10: track 0.00 -> 10.3 mm
- net N$43: track 0.00 -> 7.93 mm
- net N$29: track 0.00 -> 5.94 mm
- net MON: track 0.00 -> 5.61 mm
- net N$13: track 66.4 -> 62.3 mm
- net N$25: track 0.00 -> 3.92 mm
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
Commit message: .
Parts:
- 2R8: value 68k *80ruw -> 68k *80khz
- 2VD4: value (none) -> 22v
- 4C1: value (none) -> 100n
- moved 1TH1 29.1 mm to (40.0, 79.4)
- moved 1RZ1 23.7 mm to (41.9, 85.7), turned to 270 degrees
- moved 1R1 10.6 mm to (64.1, 76.8)
- moved 1F1 7.24 mm to (52.7, 95.2), turned to 0 degrees
- moved 2R12 6.75 mm to (61.0, 22.2), turned to 270 degrees
- moved 3VD1 4.45 mm to (48.3, 7.62), turned to 270 degrees
- moved 1C1 3.17 mm to (60.3, 84.5)
- moved 1VD4 2.54 mm to (37.5, 64.8)
- moved 2R13 2.54 mm to (68.6, 26.7)
- moved 3R6 2.01 mm to (85.7, 51.4)
- moved 1C2 1.91 mm to (48.9, 68.6)
- moved 2VD2 1.91 mm to (27.3, 45.7)
- moved 2R14 1.42 mm to (77.5, 27.3), turned to 270 degrees
- moved 2VT1 1.42 mm to (38.7, 38.1)
- moved 2R3 1.27 mm to (23.5, 62.9)
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Connections:
- net N$9 renamed +16IN
- removed net N$36: 1F1.2A, 1TH1.1
- new net N$9: 1TH1.1, PCB.SW1
- net N$32: now also 1TH1.2; no longer PCB.SW1
- net N$33: now also 1F1.2A; no longer 1TH1.2
Routing:
- net GND: track 277.0 -> 330.3 mm, vias 0 -> 2
- net N$32: track 74.3 -> 28.1 mm
- net N$9: track 0.00 -> 28.3 mm
- net N$33: track 26.4 -> 49.5 mm
- net N$18: track 7.13 -> 19.5 mm
- net N$13: track 62.3 -> 56.6 mm
- net N$44: track 47.7 -> 42.3 mm
- net N$14: track 6.81 -> 11.3 mm
- net N$36: track 3.89 -> 0.00 mm
- net +16IN: track 34.3 -> 31.3 mm
- net -IN: track 152.3 -> 150.1 mm
- net N$20: track 15.6 -> 13.5 mm
- net N$43: track 7.93 -> 6.24 mm
- net N$40: track 27.0 -> 25.5 mm
- net N$17: track 45.4 -> 44.0 mm
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
Commit message: .
Parts:
- removed 1VD1B: S1WBS60, rectifier:B-DIL
- removed 4R2: 4k7, rcl:R1206
- added 4C3A: (no value), rcl:C1812
- 4R3: value 4k7 -> 270k
- 4VD3: value (none) -> LL4148
- moved 4VD3 19.9 mm to (86.4, 65.1), turned to 90 degrees
- moved 4R3 6.38 mm to (88.9, 64.8), turned to 270 degrees
- moved 3L2 5.71 mm to (81.9, 49.5), turned to 90 degrees
- moved 3C3 4.26 mm to (85.7, 59.1)
- moved 4R6 3.38 mm to (94.3, 72.7), turned to 270 degrees
- moved 3R6 3.18 mm to (85.7, 48.3)
- moved 4VT1 2.22 mm to (101.3, 74.3)
- moved 1F1 1.91 mm to (54.6, 95.2)
- moved 4C3 1.91 mm to (88.3, 73.7), turned to 90 degrees
- moved 4R5 0.95 mm to (97.5, 72.7), turned to 270 degrees
- moved 1RZ1 0.64 mm to (41.9, 86.4)
- moved 3VD2 0.64 mm to (51.4, 21.6)
- moved 2C3 0.63 mm to (47.0, 39.4)
- moved 2R16 0.63 mm to (80.6, 19.7)
- moved 4R4 0.63 mm to (96.5, 76.8)
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Connections:
- removed net N$31: 4DD1.6, 4R2.1, 4R3.2
- net +5V: now also 4R3.2, 4VD3.C; no longer 4C3.+
- net -IN: no longer 1VD1B.-
- net GND: now also 4C3.-, 4C3A.2; no longer 4R3.1, 4VD3.A
- net N$15: no longer 1VD1B.AC2
- net N$17: now also 2T1.3; no longer 2T1.4
- net N$23: no longer 1VD1B.+
- net N$35: now also 4C3.+, 4C3A.1, 4DD1.6, 4R3.1, 4VD3.A; no longer 4C3.-, 4R2.2, 4VD3.C
- net N$44: no longer 1VD1B.AC1
Routing:
- net N$31: track 20.5 -> 0.00 mm
- net GND: track 330.3 -> 338.1 mm
- net N$13: track 56.6 -> 49.7 mm
- net N$18: track 19.5 -> 25.8 mm
- net N$17: track 44.0 -> 39.5 mm
- net +5V: track 75.4 -> 79.7 mm
- net N$33: track 49.5 -> 53.9 mm
- net N$43: track 6.24 -> 3.18 mm
- net N$35: track 20.7 -> 23.6 mm
- net -IN: track 150.1 -> 147.3 mm
- net N$15: track 49.9 -> 47.3 mm
- net N$7: track 19.4 -> 21.4 mm
- net N$42: track 21.8 -> 20.0 mm
- net MON: track 5.61 -> 7.00 mm
- net N$29: track 5.94 -> 7.05 mm
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