File: fz10_pow.brd (EAGLE design)
At the start: 107 x 100 mm, 83 parts

Commit message: .
Parts:
- removed 2R11A, 2R11B, 2R11C, 2R11D: 1, rcl:R0805
- added 2R11: (no value), rcl:P0613/15
- 2VD1: device diode:DO35-7 -> diode:DO35-10
- moved 2R9 4.45 mm to (43.2, 50.2)
- moved 3VD3 2.56 mm to (104.8, 51.8)
- moved 2C3 2.01 mm to (48.9, 38.7), turned to 0 degrees
- moved 2C6 1.91 mm to (54.0, 36.2)
- moved 2VT1 1.91 mm to (38.7, 40.0)
- moved J5V 1.91 mm to (92.1, 60.3)
- moved 2C11 1.90 mm to (33.0, 21.6), turned to 270 degrees
- moved 2R4 0.63 mm to (45.7, 31.1)
- moved 2VD1 0.63 mm to (37.5, 27.3)
- moved 2VD2 0.63 mm to (27.3, 46.4)
- moved 2VD3 0.63 mm to (43.2, 47.6)
- moved 4R5 0.32 mm to (97.5, 73.0)
Connections:
- removed net N$21: 2R11A.2, 2R11B.2, 2VT1.3
- net -IN: now also 2R11.1; no longer 2R11C.1, 2R11D.1
- net N$37: now also 2R11.2, 2VT1.3; no longer 2R11A.1, 2R11B.1, 2R11C.2, 2R11D.2
Routing:
- net N$21: track 9.58 -> 0.00 mm
- net N$31: track 0.00 -> 7.94 mm
- net +5V: track 79.7 -> 74.5 mm
- net GND: track 338.1 -> 334.2 mm
- net N$17: track 39.5 -> 35.9 mm
- net N$36: track 0.00 -> 2.86 mm
- net N$38: track 30.6 -> 33.4 mm
- net N$37: track 7.63 -> 5.07 mm
- net N$22: track 4.45 -> 3.17 mm
- net N$24: track 10.8 -> 9.53 mm
- net +16IN: track 30.8 -> 29.6 mm
- net N$35: track 23.6 -> 22.8 mm
- net -IN: track 147.3 -> 146.6 mm

Commit message: .
Parts:
- 2C11: device rcl:C050-025X075 -> rcl:C075-032X103
- moved 2C11 1.27 mm to (33.0, 20.3)
Routing:
- net GND: track 334.2 -> 333.4 mm
- net N$5: track 51.8 -> 51.0 mm
- net N$13: track 49.6 -> 49.0 mm
Changed lines of the file:
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@@
 <attribute name="VALUE" x="48.26" y="29.845" size="1.27" layer="27" rot="R90"/>
 </element>
-<element name="2C11" library="rcl" package="C050-025X075" value="4n7" x="33.02" y="21.59" smashed="yes" rot="R270">
-<attribute name="NAME" x="35.26086875" y="20.682953125" size="1.27" layer="25" ratio="10" rot="R270"/>
-<attribute name="VALUE" x="35.351128125" y="24.492953125" size="1.27" layer="27" ratio="10" rot="R270"/>
+<element name="2C11" library="rcl" package="C075-032X103" value="4n7" x="33.02" y="20.32" smashed="yes" rot="R270">
+<attribute name="NAME" x="35.26086875" y="19.412953125" size="1.27" layer="25" ratio="10" rot="R270"/>
+<attribute name="VALUE" x="35.351128125" y="23.222953125" size="1.27" layer="27" ratio="10" rot="R270"/>
 </element>
 <element name="1F1" library="fuse" package="SHK20L" value="" x="54.61" y="95.25" smashed="yes">
@@
 <wire x1="3.24" y1="8.78" x2="3.175" y2="8.845" width="1.27" layer="16"/>
 <wire x1="102.235" y1="59.055" x2="104.775" y2="55.5625" width="1.27" layer="16"/>
-<wire x1="40.64" y1="14.605" x2="48.895" y2="14.605" width="2.54" layer="16"/>
+<wire x1="42.545" y1="14.605" x2="48.895" y2="14.605" width="2.54" layer="16"/>
 <wire x1="48.895" y1="14.605" x2="50.165" y2="13.97" width="2.54" layer="16"/>
 <wire x1="50.165" y1="13.97" x2="53.6575" y2="13.97" width="2.54" layer="16"/>
 <wire x1="53.6575" y1="13.97" x2="61.2775" y2="17.145" width="2.54" layer="16"/>
-<wire x1="40.64" y1="14.605" x2="33.02" y2="6.985" width="2.54" layer="16"/>
 <wire x1="33.02" y1="6.985" x2="31.115" y2="5.08" width="1.4224" layer="16"/>
 <wire x1="31.115" y1="5.08" x2="24.765" y2="5.08" width="1.4224" layer="16"/>
@@
 <wire x1="3.175" y1="8.845" x2="3.175" y2="12.7" width="1.6764" layer="16"/>
 <wire x1="3.175" y1="12.7" x2="23.24" y2="12.7" width="1.6764" layer="16"/>
-<wire x1="23.24" y1="12.7" x2="26.035" y2="12.7" width="1.6764" layer="16"/>
 <wire x1="23.24" y1="8.78" x2="23.24" y2="12.7" width="1.6764" layer="16"/>
-<wire x1="26.035" y1="12.7" x2="33.02" y2="19.05" width="1.6764" layer="16"/>
 <wire x1="91.44" y1="80.1116" x2="91.44" y2="78.74" width="0.6096" layer="16"/>
 <wire x1="91.44" y1="78.74" x2="91.1225" y2="78.4225" width="0.6096" layer="16"/>
@@
 <wire x1="97.8154" y1="58.8772" x2="102.235" y2="58.8772" width="1.27" layer="16"/>
 <wire x1="102.235" y1="58.8772" x2="102.235" y2="59.055" width="1.27" layer="16"/>
+<wire x1="42.545" y1="14.605" x2="34.925" y2="6.985" width="2.54" layer="16"/>
+<wire x1="34.925" y1="6.985" x2="33.02" y2="6.985" width="2.54" layer="16"/>
+<wire x1="33.02" y1="16.51" x2="27.05" y2="16.51" width="1.778" layer="16"/>
+<wire x1="27.05" y1="16.51" x2="23.24" y2="12.7" width="1.778" layer="16"/>
 </signal>
 <signal name="N$19">
@@
 <contactref element="3C2" pad="+"/>
 <contactref element="3L2" pad="1"/>
-<wire x1="58.42" y1="27.94" x2="58.268" y2="27.94" width="1.27" layer="16"/>
-<wire x1="53.975" y1="21.59" x2="58.42" y2="20.955" width="1.4224" layer="16"/>
-<wire x1="58.268" y1="27.94" x2="58.268" y2="21.107" width="1.4224" layer="16"/>
 <wire x1="81.915" y1="45.72" x2="78.585921875" y2="40.485921875" width="2.1844" layer="16"/>
 <wire x1="78.585921875" y1="40.485921875" x2="76.835" y2="36.195" width="2.1844" layer="16"/>
-<wire x1="58.268" y1="21.107" x2="58.42" y2="20.955" width="1.27" layer="16"/>
-<wire x1="58.42" y1="20.955" x2="60.96" y2="20.803" width="1.27" layer="16"/>
 <wire x1="65.253" y1="20.803" x2="60.96" y2="20.803" width="1.4224" layer="16"/>
 <wire x1="65.253" y1="20.803" x2="69.215" y2="24.765" width="1.4224" layer="16"/>
 <wire x1="69.215" y1="24.765" x2="69.215" y2="28.575" width="1.4224" layer="16"/>
 <wire x1="69.215" y1="28.575" x2="76.835" y2="36.195" width="1.4224" layer="16"/>
+<wire x1="53.975" y1="21.59" x2="58.42" y2="21.59" width="1.778" layer="16"/>
+<wire x1="58.42" y1="21.59" x2="58.42" y2="27.94" width="1.778" layer="16"/>
+<wire x1="60.96" y1="20.803" x2="59.207" y2="20.803" width="1.27" layer="16"/>
+<wire x1="59.207" y1="20.803" x2="58.42" y2="21.59" width="1.27" layer="16"/>
 </signal>
 <signal name="N$14">
@@
 <contactref element="3VD1" pad="A1"/>
 <contactref element="2T1" pad="10"/>
-<wire x1="41.91" y1="10.16" x2="41.91" y2="5.08" width="1.27" layer="16"/>
 <wire x1="33.655" y1="2.54" x2="22.225" y2="2.54" width="1.4224" layer="16"/>
 <wire x1="33.655" y1="2.54" x2="39.37" y2="2.54" width="2.54" layer="16"/>
@@
 <wire x1="8.255" y1="8.765" x2="8.24" y2="8.78" width="2.54" layer="16"/>
 <wire x1="45.72" y1="5.08" x2="41.91" y2="5.08" width="1.27" layer="16"/>
-<wire x1="45.72" y1="10.16" x2="41.91" y2="10.16" width="1.27" layer="16"/>
+<wire x1="45.72" y1="10.16" x2="43.18" y2="10.16" width="1.27" layer="16"/>
+<wire x1="43.18" y1="10.16" x2="41.91" y2="8.89" width="1.27" layer="16"/>
+<wire x1="41.91" y1="8.89" x2="41.91" y2="5.08" width="1.27" layer="16"/>
 </signal>
 <signal name="N$28">
@@
 <contactref element="3VD2" pad="A1"/>
 <contactref element="2T1" pad="6"/>
-<wire x1="28.24" y1="8.78" x2="38.51" y2="19.05" width="2.54" layer="16"/>
-<wire x1="49.53" y1="19.05" x2="49.8475" y2="18.7325" width="1.6764" layer="16"/>
-<wire x1="49.8475" y1="18.7325" x2="50.165" y2="19.05" width="1.6764" layer="16"/>
-<wire x1="50.165" y1="19.05" x2="53.975" y2="19.05" width="1.6764" layer="16"/>
-<wire x1="38.51" y1="19.05" x2="49.53" y2="19.05" width="2.54" layer="16"/>
-<wire x1="53.975" y1="24.13" x2="51.435" y2="23.495" width="1.27" layer="16"/>
-<wire x1="51.435" y1="23.495" x2="50.165" y2="22.86" width="1.27" layer="16"/>
-<wire x1="50.165" y1="22.86" x2="50.165" y2="19.685" width="1.27" layer="16"/>
-<wire x1="50.165" y1="19.685" x2="49.8475" y2="18.7325" width="1.27" layer="16"/>
+<wire x1="49.53" y1="19.05" x2="53.975" y2="19.05" width="1.6764" layer="16"/>
+<wire x1="53.975" y1="24.13" x2="50.8" y2="24.13" width="1.27" layer="16"/>
+<wire x1="50.8" y1="24.13" x2="49.53" y2="22.86" width="1.27" layer="16"/>
+<wire x1="49.53" y1="22.86" x2="49.53" y2="19.685" width="1.27" layer="16"/>
+<wire x1="49.53" y1="19.05" x2="40.64" y2="19.05" width="2.54" layer="16"/>
+<wire x1="40.64" y1="19.05" x2="33.655" y2="12.065" width="2.54" layer="16"/>
+<wire x1="33.655" y1="12.065" x2="31.525" y2="12.065" width="2.54" layer="16"/>
+<wire x1="31.525" y1="12.065" x2="28.24" y2="8.78" width="2.54" layer="16"/>
+<wire x1="49.53" y1="19.05" x2="49.53" y2="19.685" width="1.778" layer="16"/>
 </signal>
 <signal name="N$39">

Commit message: .
Parts:
- 2C2: device rcl:C050-025X075 -> rcl:C075-032X103
- moved 2C2 4.49 mm to (26.7, 52.1), turned to 20 degrees
- moved 2R7 3.86 mm to (67.9, 44.5)
- moved 2C7 3.86 mm to (67.3, 50.8)
- moved 2VD2 3.86 mm to (27.9, 42.5)
- moved 4R5 1.91 mm to (97.5, 71.1)
- moved 4VT1 1.91 mm to (101.3, 72.4)
- moved 2C4 1.80 mm to (65.4, 40.6)
- moved 2VT1 1.42 mm to (37.5, 40.6)
- moved 2R10 1.27 mm to (66.7, 48.3)
- moved 2R1 1.27 mm to (34.9, 57.8), turned to 172 degrees
- moved 4R6 1.27 mm to (94.3, 71.4)
- moved 4VD3 1.14 mm to (85.7, 64.1)
- moved 4R3 1.14 mm to (88.3, 63.8)
- moved 4C1 1.00 mm to (102.6, 83.2), turned to 180 degrees
- moved 2VD4 0.64 mm to (48.3, 53.3)
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Connections:
- net -IN: now also 2T1.3; no longer 2T1.2
- net N$17: now also 2T1.2; no longer 2T1.3
Routing:
- net -IN: track 146.6 -> 168.2 mm
- net N$30: track 5.68 -> 12.6 mm
- net N$17: track 35.9 -> 29.1 mm, vias 2 -> 0
- net N$40: track 25.5 -> 20.8 mm
- net N$23: track 70.1 -> 72.8 mm
- net +16IN: track 29.6 -> 31.1 mm
- net N$4: track 6.59 -> 8.04 mm
- net MON: track 7.00 -> 5.73 mm
- net N$6: track 7.00 -> 5.84 mm
- net N$32: track 28.6 -> 29.4 mm
- net N$35: track 22.8 -> 23.6 mm
- net GND: track 333.4 -> 334.0 mm
- net +5V: track 74.5 -> 75.1 mm, vias 2 -> 0
- net N$20: track 13.5 -> 12.9 mm
- net N$37: track 5.07 -> 5.62 mm

Commit message: .
Parts:
- 2VD1: device diode:DO35-10 -> diode:SOD80C
- moved 2R11 9.09 mm to (32.4, 40.6), turned to 270 degrees
- moved 2R4 8.78 mm to (37.1, 29.2), turned to 180 degrees
- moved 2VD1 8.72 mm to (28.9, 28.9), flipped to the bottom, turned to 0 degrees
- moved 1VD1 7.10 mm to (29.2, 73.7), turned to 0 degrees
- moved 2C2 5.40 mm to (29.2, 56.8), turned to 270 degrees
- moved 1VD4 5.09 mm to (42.5, 65.1)
- moved 1VD3 4.97 mm to (38.1, 69.5)
- moved 2R3 4.14 mm to (23.8, 58.7)
- moved 2R1 3.13 mm to (36.2, 60.6), turned to 135 degrees
- moved 1VD2 2.84 mm to (29.2, 69.8), turned to 0 degrees
- moved 2C11 1.27 mm to (33.0, 21.6)
- moved 2VD2 0.32 mm to (27.6, 42.5)
Routing:
- net N$44: track 42.3 -> 29.1 mm
- net -IN: track 168.2 -> 156.4 mm
- net +16IN: track 31.1 -> 38.3 mm
- net N$24: track 9.63 -> 5.03 mm
- net N$23: track 72.8 -> 70.0 mm
- net N$15: track 47.3 -> 45.0 mm
- net N$30: track 12.6 -> 10.4 mm
- net N$37: track 5.62 -> 7.18 mm

Commit message: .
Parts:
- moved 2R4 2.29 mm to (38.4, 31.1)
- moved 2R11 1.59 mm to (32.4, 42.2)
- moved 3C2 1.59 mm to (79.4, 34.6)
- moved 2VD1 1.42 mm to (29.5, 30.2)
- moved 3L2 1.27 mm to (81.9, 48.3)
- moved 2VD2 1.27 mm to (27.6, 43.8)
- moved 2C11 0.95 mm to (33.0, 22.5)
- moved 1L1 0.64 mm to (64.8, 65.4)
- moved 2R16 0.32 mm to (80.6, 20.0)
Routing:
- net -IN: track 156.4 -> 153.7 mm
- net +16IN: track 38.3 -> 35.7 mm
- net GND: track 334.4 -> 336.6 mm
- net N$17: track 29.1 -> 27.3 mm
- net N$24: track 5.03 -> 6.34 mm
- net N$30: track 10.4 -> 9.11 mm
- net N$37: track 7.18 -> 6.16 mm
- net N$22: track 2.76 -> 3.51 mm
- net N$32: track 29.4 -> 30.0 mm
- net N$33: track 53.9 -> 54.5 mm

Commit message: .
Parts:
- 2R10: value 1k -> 470
- 2R11: value (none) -> 1
- 2VD1: value 1N4148 -> LL4148
- moved 2C11 2.54 mm to (33.0, 20.0)
- moved 1VD1 1.42 mm to (30.5, 74.3)
- moved 1VD2 1.42 mm to (30.5, 69.2)
- moved 3VD1 1.27 mm to (48.3, 8.89)
- moved 2VT1 1.27 mm to (38.7, 40.6)
- moved 1VD3 0.90 mm to (38.7, 70.2)
- moved 2R1 0.90 mm to (36.8, 61.3)
- moved 1C2 0.64 mm to (48.9, 69.2)
- moved 1VD4 0.63 mm to (42.5, 65.7)
Routing:
- net N$23: track 70.0 -> 73.0 mm
- net N$17: track 27.3 -> 28.6 mm
- net GND: track 336.6 -> 335.4 mm
- net N$44: track 29.2 -> 28.1 mm
- net N$37: track 6.16 -> 7.25 mm
- net N$39: track 64.7 -> 63.8 mm
- net N$11: track 7.77 -> 7.09 mm
- net N$28: track 38.7 -> 39.4 mm
- net N$5: track 51.0 -> 51.6 mm
- added copper zone on layer 16, net N$17

Commit message: .
Parts:
- added 2R4B: (no value), rcl:0207/10
- 2C11: value 4n7 -> 4n7 1kv
- 2R10: device rcl:R1206 -> rcl:0207/10
- 2R11: value 1 -> 0.91e
- 2R4: device rcl:0204/7 -> rcl:M0805
- 2R7: device rcl:R1206 -> rcl:R0805
- 2R8: value 68k *80khz -> 68k *(80khz); device rcl:R1206 -> rcl:R0805
- 2VD4: value 22v -> 22v(1n4748a)
- 3R5A: value 82k -> 30k
- 3R5B: value (none) -> 56k
- 3R5C: value (none) -> 560
- 3R6B: value 0 -> 0jp
- 3VD3: value 12v -> 12v(1n4742a)
- 4C1: device rcl:C1206 -> rcl:C0805
- moved 2R10 21.2 mm to (50.2, 34.9), flipped to the top
- moved 2C3 8.64 mm to (46.4, 30.5), turned to 315 degrees
- moved 2C6 5.85 mm to (50.2, 31.8)
- moved 2R8 2.84 mm to (54.0, 39.4), turned to 0 degrees
- moved 2C7 2.01 mm to (67.9, 48.9)
- moved 2VD1 1.27 mm to (28.3, 30.2)
- moved 1TH1 0.64 mm to (39.4, 79.4)
- moved 2R4 0.63 mm to (37.8, 31.1), flipped to the bottom, turned to 0 degrees
- moved 2R7 0.63 mm to (67.9, 45.1), turned to 0 degrees
Connections:
- removed net N$37: 2R11.2, 2VT1.3
- new net N$21: 2R10.2, 2R11.2, 2VT1.3
- net +16IN: now also 2R4B.1
- net -IN: no longer 2R10.2
- net N$22: now also 2R4B.2
Routing:
- net N$21: track 0.00 -> 16.2 mm
- net N$4: track 8.04 -> 21.6 mm
- net -IN: track 154.1 -> 145.7 mm
- net N$20: track 12.9 -> 20.7 mm
- net N$37: track 7.25 -> 0.00 mm
- net +16IN: track 35.9 -> 41.1 mm
- net N$22: track 3.51 -> 7.07 mm
- net N$3: track 14.0 -> 17.2 mm
- net N$40: track 20.8 -> 22.1 mm
- net N$24: track 6.34 -> 5.50 mm
- net N$9: track 28.4 -> 27.8 mm
Other:
- board text added: "REV1.1"
- board text removed: "REV1.0"

Commit message: .
Parts:
- 3VD3: value 12v(1n4742a) -> 12v(1N4742A)
- 4DD1: value 4011D -> CD4011BM
- 4R1C: value (none) -> 200k
- moved 2R4 3.86 mm to (34.0, 30.5)
- moved 2R4B 3.24 mm to (34.3, 30.5)
- moved 2VD1 2.69 mm to (26.4, 28.3), turned to 270 degrees
- moved 2C3 0.64 mm to (47.0, 30.5)
- moved 2C6 0.63 mm to (50.8, 31.8)
- moved 2VT1 0.63 mm to (38.7, 40.0)
Routing:
- net +16IN: track 41.1 -> 45.5 mm
- net N$24: track 5.50 -> 3.21 mm
- net N$21: track 16.2 -> 15.6 mm
- net N$11: track 7.09 -> 7.72 mm
- net -IN: track 145.7 -> 146.2 mm
