File: fz10_pow.brd (EAGLE design)
At the start: 107 x 100 mm, 81 parts

Commit message: .
Parts:
- removed 4C3A: (no value), rcl:C1812
- added 4C3B: (no value), rcl:E2,5-5
- 2VT1: value IRF3704L-V -> 2SK1984
- 3VD1: value BYV32 -> FCB06A06
- 3VD2: value BYV32 -> MA10799
- 4C3: value 4m7 -> 10m; device rcl:E2,5-5 -> rcl:C1812
- moved 4C3 5.28 mm to (83.8, 70.8), flipped to the bottom
Connections:
- net GND: now also 4C3.2, 4C3B.-; no longer 4C3.-, 4C3A.2
- net N$35: now also 4C3.1, 4C3B.+; no longer 4C3.+, 4C3A.1
Other:
- board text added: "220V"

Commit message: .
Parts:
- moved 2R8 0.63 mm to (53.3, 39.4)
- renumbered 4C2C to 4C2B, 4C3 to 4C3A
Routing:
- net N$20: track 20.4 -> 19.4 mm
- net N$3: track 17.2 -> 17.8 mm
Changed lines of the file:
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@@
 <attribute name="VALUE" x="104.4575" y="78.74" size="1.27" layer="28" rot="MR0"/>
 </element>
-<element name="4C2C" library="rcl" package="C1206" value="" x="84.455" y="93.345" smashed="yes" rot="MR90">
+<element name="4C2B" library="rcl" package="C1206" value="" x="84.455" y="93.345" smashed="yes" rot="MR90">
 <attribute name="NAME" x="85.725" y="92.075" size="1.27" layer="26" rot="MR180"/>
 <attribute name="VALUE" x="81.915" y="92.075" size="1.27" layer="28" rot="MR90"/>
@@
 <attribute name="NAME" x="56.3245" y="31.6865" size="1.27" layer="25" ratio="10" rot="R180"/>
 </element>
-<element name="2R8" library="rcl" package="R0805" value="68k *(80khz)" x="53.975" y="39.37" smashed="yes" rot="MR0">
-<attribute name="NAME" x="50.165" y="42.545" size="1.27" layer="26" rot="MR0"/>
-<attribute name="VALUE" x="50.165" y="40.64" size="1.27" layer="28" rot="MR0"/>
+<element name="2R8" library="rcl" package="R0805" value="68k *(80khz)" x="53.34" y="39.37" smashed="yes" rot="MR0">
+<attribute name="NAME" x="49.53" y="42.545" size="1.27" layer="26" rot="MR0"/>
+<attribute name="VALUE" x="49.53" y="40.64" size="1.27" layer="28" rot="MR0"/>
 </element>
 <element name="2C6" library="rcl" package="C0805" value="100n" x="50.8" y="31.75" smashed="yes" rot="MR0">
@@
 <attribute name="VALUE" x="58.1025" y="83.5025" size="1.27" layer="27" rot="R180"/>
 </element>
-<element name="4C3" library="rcl" package="C1812" value="10m" x="83.82" y="70.8025" smashed="yes" rot="MR90">
+<element name="4C3A" library="rcl" package="C1812" value="10m" x="83.82" y="70.8025" smashed="yes" rot="MR90">
 <attribute name="NAME" x="81.28" y="73.025" size="1.27" layer="26" rot="MR270"/>
 <attribute name="VALUE" x="80.01" y="68.8975" size="1.27" layer="28" rot="MR90"/>
@@
 <contactref element="4R1C" pad="3"/>
 <contactref element="4VD1" pad="A"/>
-<contactref element="4C2C" pad="2"/>
+<contactref element="4C2B" pad="2"/>
 <contactref element="4R1A" pad="1"/>
 <wire x1="84.455" y1="86.1945" x2="88.265" y2="84.455" width="0.8128" layer="16"/>
@@
 <contactref element="4C3B" pad="-"/>
 <wire x1="88.265" y1="74.93" x2="91.1225" y2="78.4225" width="0.8128" layer="16"/>
-<contactref element="4C3" pad="2"/>
+<contactref element="4C3A" pad="2"/>
 <wire x1="83.82" y1="72.7525" x2="83.82" y2="74.93" width="1.27" layer="16"/>
 <wire x1="83.82" y1="74.93" x2="88.265" y2="74.93" width="1.27" layer="16"/>
@@
 <contactref element="4DD1" pad="2"/>
 <contactref element="4C2A" pad="1"/>
-<contactref element="4C2C" pad="1"/>
+<contactref element="4C2B" pad="1"/>
 <wire x1="99.06" y1="80.1116" x2="99.06" y2="82.2325" width="0.4064" layer="16"/>
 <wire x1="99.06" y1="82.2325" x2="97.79" y2="82.2325" width="0.4064" layer="16"/>
@@
 <contactref element="2R8" pad="2"/>
 <contactref element="1PC1" pad="4"/>
-<wire x1="53.025" y1="39.37" x2="52.705" y2="39.055" width="0.6096" layer="16"/>
-<wire x1="52.705" y1="39.055" x2="52.705" y2="41.91" width="0.6096" layer="16"/>
 <wire x1="58.42" y1="35.56" x2="58.42" y2="34.29" width="1.016" layer="16"/>
 <wire x1="58.42" y1="34.29" x2="56.515" y2="32.385" width="1.016" layer="16"/>
@@
 <wire x1="51.75" y1="31.75" x2="51.5925" y2="34.7675" width="1.016" layer="16"/>
 <wire x1="51.75" y1="31.75" x2="52.385" y2="32.385" width="1.016" layer="16"/>
-<wire x1="53.025" y1="39.37" x2="51.5925" y2="37.3025" width="1.016" layer="16"/>
+<wire x1="52.39" y1="39.37" x2="51.5925" y2="37.3025" width="1.016" layer="16"/>
 <wire x1="51.5925" y1="37.3025" x2="51.5925" y2="34.7675" width="1.016" layer="16"/>
+<wire x1="52.39" y1="39.37" x2="52.39" y2="41.595" width="0.8128" layer="16"/>
+<wire x1="52.39" y1="41.595" x2="52.705" y2="41.91" width="0.8128" layer="16"/>
 </signal>
 <signal name="N$3">
@@
 <contactref element="2C5" pad="1"/>
 <wire x1="60.325" y1="49.53" x2="61.595" y2="52.705" width="1.6764" layer="16"/>
-<wire x1="54.925" y1="39.37" x2="55.88" y2="40.6425" width="0.6096" layer="16"/>
-<wire x1="55.88" y1="40.6425" x2="55.88" y2="47.625" width="0.6096" layer="16"/>
+<wire x1="55.88" y1="40.64" x2="55.88" y2="47.625" width="0.6096" layer="16"/>
 <wire x1="55.88" y1="47.625" x2="57.785" y2="49.53" width="0.6096" layer="16"/>
 <wire x1="57.785" y1="49.53" x2="60.325" y2="49.53" width="0.6096" layer="16"/>
+<wire x1="55.88" y1="40.64" x2="54.61" y2="39.37" width="0.6096" layer="16"/>
+<wire x1="54.61" y1="39.37" x2="54.29" y2="39.37" width="0.6096" layer="16"/>
 </signal>
 <signal name="-IN">
@@
 <wire x1="92.71" y1="76.2" x2="89.535" y2="72.39" width="0.8128" layer="16"/>
 <wire x1="89.535" y1="72.39" x2="88.265" y2="72.39" width="0.8128" layer="16"/>
-<contactref element="4C3" pad="1"/>
+<contactref element="4C3A" pad="1"/>
 <wire x1="85.725" y1="65.835" x2="87.3125" y2="65.835" width="1.27" layer="16"/>
 <wire x1="87.3125" y1="65.835" x2="87.63" y2="65.835" width="1.27" layer="16"/>

Commit message: .
Parts:
- added 2C12: 100n, rcl:C0805
- 2R16: value 3k3 -> 10k
- 4VD2: value LL4158 -> LL4148
Connections:
- net +16IN: now also 2C12.1
- net -IN: now also 2C12.2
Routing:
- net -IN: track 146.2 -> 147.2 mm
- net +16IN: track 45.5 -> 46.5 mm
Changed lines of the file:
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@@
 <attribute name="VALUE" x="75.057" y="82.6135" size="1.27" layer="28" rot="MR90"/>
 </element>
-<element name="4VD2" library="diode" package="SOD80C" value="LL4158" x="81.915" y="79.6925" smashed="yes" rot="MR270">
+<element name="4VD2" library="diode" package="SOD80C" value="LL4148" x="81.915" y="79.6925" smashed="yes" rot="MR270">
 <attribute name="NAME" x="77.343" y="76.2635" size="1.27" layer="26" rot="MR90"/>
 <attribute name="VALUE" x="76.708" y="81.2165" size="1.27" layer="28" rot="MR270"/>
@@
 <attribute name="VALUE" x="79.756" y="25.146" size="1.27" layer="27" ratio="10"/>
 </element>
-<element name="2R16" library="rcl" package="R1206" value="3k3" x="80.645" y="20.0025" smashed="yes" rot="MR90">
+<element name="2R16" library="rcl" package="R1206" value="10k" x="80.645" y="20.0025" smashed="yes" rot="MR90">
 <attribute name="NAME" x="82.55" y="21.9075" size="1.27" layer="26" rot="MR180"/>
 <attribute name="VALUE" x="82.55" y="20.0025" size="1.27" layer="28" rot="MR180"/>
@@
 </element>
 <element name="2R4B" library="rcl" package="0207/10" value="" x="34.29" y="30.48" rot="R180"/>
+<element name="2C12" library="rcl" package="C0805" value="100n" x="43.815" y="28.575" smashed="yes" rot="MR270">
+<attribute name="NAME" x="41.91" y="25.4" size="1.27" layer="26" rot="MR0"/>
+<attribute name="VALUE" x="46.355" y="29.845" size="1.27" layer="28" rot="MR270"/>
+</element>
 </elements>
 <signals>
@@
 <wire x1="40.16375" y1="63.02375" x2="38.735" y2="65.0875" width="2.54" layer="16"/>
 <wire x1="40.16375" y1="62.07125" x2="40.16375" y2="63.02375" width="2.54" layer="16"/>
-<wire x1="44.341053125" y1="26.67" x2="35.8775" y2="26.67" width="1.4224" layer="16"/>
+<wire x1="44.341053125" y1="26.67" x2="43.815" y2="26.67" width="1.4224" layer="16"/>
+<wire x1="43.815" y1="26.67" x2="35.8775" y2="26.67" width="1.4224" layer="16"/>
 <wire x1="35.8775" y1="26.67" x2="33.02" y2="23.8125" width="1.4224" layer="16"/>
 <wire x1="68.895" y1="45.085" x2="69.85" y2="45.085" width="1.27" layer="16"/>
@@
 <wire x1="47.888025" y1="29.581971875" x2="49.215" y2="31.543946875" width="1.27" layer="16"/>
 <wire x1="49.215" y1="31.543946875" x2="49.85" y2="31.75" width="1.27" layer="16"/>
+<contactref element="2C12" pad="2"/>
+<wire x1="43.815" y1="27.625" x2="43.815" y2="26.67" width="0.6096" layer="16"/>
 </signal>
 <signal name="N$4">
@@
 <wire x1="46.091971875" y1="31.378025" x2="47.625" y2="33.546053125" width="1.27" layer="16"/>
 <wire x1="47.625" y1="33.546053125" x2="47.625" y2="44.45" width="1.27" layer="16"/>
-<wire x1="39.37" y1="30.48" x2="45.193946875" y2="30.48" width="1.27" layer="16"/>
+<wire x1="39.37" y1="30.48" x2="43.815" y2="30.48" width="1.27" layer="16"/>
+<wire x1="43.815" y1="30.48" x2="45.193946875" y2="30.48" width="1.27" layer="16"/>
 <wire x1="45.193946875" y1="30.48" x2="46.091971875" y2="31.378025" width="1.27" layer="16"/>
+<contactref element="2C12" pad="1"/>
+<wire x1="43.815" y1="29.525" x2="43.815" y2="30.48" width="0.6096" layer="16"/>
 </signal>
 <signal name="N$8">

Commit message: .
Parts:
- 2R16: value 10k -> 8k2
- 3R5A: value 30k -> (none)
- 3R5B: value 56k -> (none)
- 3R5C: value 560 -> (none)
- 3R6: value 3k9 -> 9k1
- 3R7: value 100 -> 82
Changed lines of the file:
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@@
 <attribute name="VALUE" x="79.756" y="25.146" size="1.27" layer="27" ratio="10"/>
 </element>
-<element name="2R16" library="rcl" package="R1206" value="10k" x="80.645" y="20.0025" smashed="yes" rot="MR90">
+<element name="2R16" library="rcl" package="R1206" value="8k2" x="80.645" y="20.0025" smashed="yes" rot="MR90">
 <attribute name="NAME" x="82.55" y="21.9075" size="1.27" layer="26" rot="MR180"/>
 <attribute name="VALUE" x="82.55" y="20.0025" size="1.27" layer="28" rot="MR180"/>
@@
 <attribute name="VALUE" x="97.7646" y="41.1226" size="1.27" layer="27" ratio="10" rot="R180"/>
 </element>
-<element name="3R7" library="rcl" package="P0613/15" value="100" x="102.235" y="51.435" smashed="yes" rot="R270">
+<element name="3R7" library="rcl" package="P0613/15" value="82" x="102.235" y="51.435" smashed="yes" rot="R270">
 <attribute name="NAME" x="100.838" y="56.0324" size="1.27" layer="25" ratio="10"/>
 <attribute name="VALUE" x="100.457" y="53.8988" size="1.27" layer="27" ratio="10"/>
 </element>
-<element name="3R5A" library="rcl" package="M1206" value="30k" x="104.14" y="36.195" smashed="yes" rot="MR90">
+<element name="3R5A" library="rcl" package="M1206" value="" x="104.14" y="36.195" smashed="yes" rot="MR90">
 <attribute name="NAME" x="105.41" y="41.275" size="1.27" layer="26" rot="MR0"/>
 <attribute name="VALUE" x="105.41" y="39.37" size="1.27" layer="28" rot="MR0"/>
 </element>
-<element name="3R5B" library="rcl" package="M1206" value="56k" x="98.425" y="34.29" smashed="yes" rot="MR180">
+<element name="3R5B" library="rcl" package="M1206" value="" x="98.425" y="34.29" smashed="yes" rot="MR180">
 <attribute name="NAME" x="95.25" y="33.02" size="1.27" layer="26" rot="MR0"/>
 <attribute name="VALUE" x="97.155" y="36.83" size="1.27" layer="28" rot="MR180"/>
 </element>
-<element name="3R5C" library="rcl" package="0207/10" value="560" x="92.075" y="31.115" smashed="yes">
+<element name="3R5C" library="rcl" package="0207/10" value="" x="92.075" y="31.115" smashed="yes">
 <attribute name="NAME" x="90.17" y="30.48" size="1.27" layer="25"/>
 <attribute name="VALUE" x="90.805" y="28.575" size="1.27" layer="27"/>
 </element>
-<element name="3R6" library="rcl" package="0204/7" value="3k9" x="85.725" y="48.26" smashed="yes" rot="R90">
+<element name="3R6" library="rcl" package="0204/7" value="9k1" x="85.725" y="48.26" smashed="yes" rot="R90">
 <attribute name="NAME" x="86.36" y="46.355" size="1.27" layer="25" rot="R90"/>
 <attribute name="VALUE" x="88.265" y="46.6725" size="1.27" layer="27" rot="R90"/>

Commit message: .
Parts:
- added 2VD5: 1N4148, diode:DO35-7
- 2R16: value 8k2 -> 8.20k
- 2VD3: value LL4148 -> 1N4148
- 3R6: value 9k1 -> 8.32k
Connections:
- new net N$45: 2VD5.A
- net N$5: now also 2VD5.C
Changed lines of the file:
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@@
 <attribute name="VALUE" x="40.64" y="52.705" size="1.27" layer="27" rot="R180"/>
 </element>
-<element name="2VD3" library="diode" package="DO35-7" value="LL4148" x="43.18" y="47.625" smashed="yes" rot="R180">
+<element name="2VD3" library="diode" package="DO35-7" value="1N4148" x="43.18" y="47.625" smashed="yes" rot="R180">
 <attribute name="NAME" x="47.371" y="46.0375" size="1.27" layer="25" ratio="10" rot="R180"/>
 <attribute name="VALUE" x="48.006" y="44.577" size="1.27" layer="27" ratio="10" rot="R180"/>
@@
 <attribute name="VALUE" x="79.756" y="25.146" size="1.27" layer="27" ratio="10"/>
 </element>
-<element name="2R16" library="rcl" package="R1206" value="8k2" x="80.645" y="20.0025" smashed="yes" rot="MR90">
+<element name="2R16" library="rcl" package="R1206" value="8.20k" x="80.645" y="20.0025" smashed="yes" rot="MR90">
 <attribute name="NAME" x="82.55" y="21.9075" size="1.27" layer="26" rot="MR180"/>
 <attribute name="VALUE" x="82.55" y="20.0025" size="1.27" layer="28" rot="MR180"/>
@@
 <attribute name="VALUE" x="90.805" y="28.575" size="1.27" layer="27"/>
 </element>
-<element name="3R6" library="rcl" package="0204/7" value="9k1" x="85.725" y="48.26" smashed="yes" rot="R90">
+<element name="3R6" library="rcl" package="0204/7" value="8.32k" x="85.725" y="48.26" smashed="yes" rot="R90">
 <attribute name="NAME" x="86.36" y="46.355" size="1.27" layer="25" rot="R90"/>
 <attribute name="VALUE" x="88.265" y="46.6725" size="1.27" layer="27" rot="R90"/>
@@
 <attribute name="VALUE" x="46.355" y="29.845" size="1.27" layer="28" rot="MR270"/>
 </element>
+<element name="2VD5" library="diode" package="DO35-7" value="1N4148" x="65.405" y="15.24"/>
 </elements>
 <signals>
@@
 <wire x1="43.18" y1="11.43" x2="41.91" y2="10.16" width="1.27" layer="16"/>
 <wire x1="41.91" y1="10.16" x2="41.91" y2="6.35" width="1.27" layer="16"/>
+<contactref element="2VD5" pad="C"/>
+<wire x1="45.72" y1="11.43" x2="61.595" y2="15.24" width="0" layer="19" extent="1-1"/>
 </signal>
 <signal name="N$28">
@@
 <wire x1="38.735" y1="37.465" x2="38.735" y2="34.925" width="2.1844" layer="16"/>
 </signal>
+<signal name="N$45">
+<contactref element="2VD5" pad="A"/>
+</signal>
 </signals>
