File: fz10_pow.sch (EAGLE design)
At the start: 71 parts, among them T1 TRANS_ER29

Commit message: .
Parts:
- removed C100: 220nx250v, 3do:C26X19
- removed C103: 470mfx25v, rcl:CPOL-EUE5-8.5
- removed C12A, C12B: (no value), rcl:C-EU050-025X075
- removed C12C, C12D, C14: (no value), rcl:C-EUC1206
- removed D1, D2, D3, D4: 1N4004, diode:1N4004
- removed DD1: 4011D, 40xx:4011D
- removed F1: (no value), fuse:SHK20L
- removed L1: LFLF-10X13, DSS0:LFLF-10X13
- removed R1, R10, R11, R11A, R11B, R17A, R17B, R18, R19, R2, R6, R7: (no value), rcl:R-EU_R1206
- removed R155A: 82k, rcl:R-EU_M1206
- removed R156: 3k9, rcl:R-EU_M1206
- removed R17: (no value), rcl:R-TRIMM3296W
- removed T2: (no value), transistor:-NPN-TO92-ECB
- removed VD6, VD7: 1N4148DO35-7, diode:1N4148DO35-7
- added 1C1: 220nX250v, 3do:C26X19
- added 1C2: 100nX250v, rcl:C-EU150-084X183
- added 1F1: (no value), fuse:SHK20L
- added 1L1: LFLF-10X13, DSS0:LFLF-10X13
- added 1R1: 470k, rcl:R-EU_0613/15
- added 1RZ1: S1210, varistor:S1210
- added 1TH1: THERMISTOR-7,5, varistor:THERMISTOR-7,5
- added 1VD1, 1VD2, 1VD3, 1VD4: 1N4007, diode:1N4004
- added 1VD1B: S1WBS60, rectifier:B-DIL
- added 2R10, 4R5: 1k, rcl:R-EU_R1206
- added 2R11A, 2R11B, 2R11C, 2R11D: 1, rcl:R-EU_R0805
- added 2R7, 4R1A, 4R1B: (no value), rcl:R-EU_R1206
- added 3C3: 470mfx25v, rcl:CPOL-EUE5-8.5
- added 3R5A: 82k, rcl:R-EU_M1206
- added 3R6: 3k9, rcl:R-EU_M1206
- added 4C1, 4C2C, 4C2D: (no value), rcl:C-EUC1206
- added 4C2A, 4C2B: (no value), rcl:C-EU050-025X075
- added 4C3: 4m7, rcl:CPOL-EUE2.5-5
- added 4DD1: 4011D, 40xx:4011D
- added 4R1C: (no value), rcl:R-TRIMM3296W
- added 4R2, 4R3: 4k7, rcl:R-EU_R1206
- added 4R4: 2k, rcl:R-EU_R1206
- added 4VD1: LL4148, diode:DIODE-SOD80C
- added 4VD2: LL4158, diode:DIODE-SOD80C
- added 4VD3: 1N4148DO35-7, diode:1N4148DO35-7
- added 4VT1: KT315, transistor:-NPN-TO92-ECB
- added J5V, J9V, JGND, JMON: (no value), pinhead:PINHD-1X1
- 2C2: value (none) -> 10n
- 2R1: value (none) -> 220k 1w
- 2R3: value (none) -> 80k 1w
- 2R4: value (none) -> 22
- renumbered C1 to 1C7, C10 to 2C10, C101 to 3C1, C102 to 3C2, C11 to 2C11, C2 to 2C2, C3 to 2C3, C4 to 2C4, C5 to 2C5, C6 to 2C6, C7 to 2C7, C8 to 3C5, D5 to 2VD4, D6 to 3VD1, D7 to 3VD2, DA1 to 1DA1, L2 to 3L1, L3 to 3L2, R1-2 to 2R1, R12 to 2R12, R13 to 2R13, R14 to 2R14, R155B to 3R5B, R155C to 3R5C, R16 to 2R16, R20 to 3R7, R3 to 2R3, R4 to 2R4, R5 to 2R5, R8 to 2R8, R9 to 2R9, T1 to 2T1, VD1 to 2VD1, VD2 to 2VD2, VD3 to 2VD3, VT1 to 2VT1
Connections:
- removed net N$38: R2.2, R6.2
- new net N$29: 1C2.2, 1L1.2, 1VD1B.AC1, 1VD2.A, 1VD4.C
- new net N$37: 2R11A.1, 2R11B.1, 2R11C.2, 2R11D.2
- net +5V: now also 3C3.+, 3R6.2, 4C1.1, 4C3.+, 4DD1P.VDD, 4R5.2, J5V.1; no longer C103.+, C14.1, DD1P.VDD, R156.2, R19.2
- net +9V: now also 3R5A.2, J9V.1; no longer R155A.2
- net -IN: now also 1VD1B.-, 1VD3.A, 1VD4.A, 2R10.2, 2R11C.1, 2R11D.1, 2R7.1; no longer D3.A, D4.A, R10.2, R11A.1, R11B.1, R7.1
- net GND: now also 3C3.-, 4C1.2, 4DD1P.VSS, 4R3.1, 4VD3.A, 4VT1.E, JGND.1; no longer C103.-, C14.2, DD1P.VSS, T2.E
- net MON: now also 4R5.1, 4VT1.C, JMON.1; no longer R19.1, T2.C
- net N$1: now also 4C2A.2, 4C2B.2, 4C2C.2, 4C2D.2, 4DD1A.I0, 4DD1A.I1, 4R1A.1, 4R1C.E, 4VD1.A; no longer C12A.2, C12B.2, C12C.2, C12D.2, DD1A.I0, DD1A.I1, R17.E, R17A.1, VD6.A
- net N$10: now also 4R1A.2, 4R1B.1, 4R1C.S, 4VD1.C, 4VD2.C; no longer R17.S, R17A.2, R17B.1, VD6.C, VD7.C
- net N$15: now also 1C2.1, 1L1.4, 1VD1.A, 1VD1B.AC2, 1VD3.C; no longer D1.A, D3.C, L1.4
- net N$18: now also 1F1.1A; no longer F1.1A
- net N$19: now also 4C2A.1, 4C2B.1, 4C2C.1, 4C2D.1, 4DD1B.O, 4DD1D.I0, 4DD1D.I1, 4R1B.2, 4R1C.A, 4VD2.A; no longer C12A.1, C12B.1, C12C.1, C12D.1, DD1B.O, DD1D.I0, DD1D.I1, R17.A, R17B.2, VD7.A
- net N$2: now also 4DD1A.O, 4DD1B.I0, 4DD1B.I1; no longer DD1A.O, DD1B.I0, DD1B.I1
- net N$21: now also 2R11A.2, 2R11B.2; no longer R11A.2, R11B.2
- net N$23: now also 1VD1.C, 1VD1B.+, 1VD2.C; no longer D1.C, D2.C
- net N$25: now also 4DD1C.O, 4R4.1; no longer DD1C.O, R18.1
- net N$26: now also 4R4.2, 4VT1.B; no longer R18.2, T2.B
- net N$27: now also 3R5A.1; no longer R155A.1
- net N$31: now also 4DD1C.I0, 4R2.1, 4R3.2; no longer R1.2, R2.1
- net N$32: now also 1C1.2, 1L1.1, 1R1.1, 1RZ1.2, PCB_SW.P; no longer C100.2, L1.3, PCB_SW.S, R11.1
- net N$33: now also 1C1.1, 1L1.3, 1R1.2, 1RZ1.1, 1TH1.2; no longer C100.1, F1.2A, L1.1, R1.1
- net N$34: now also PCB_SW.S; no longer PCB_SW.P
- net N$35: now also 4C3.-, 4R2.2, 4VD3.C; no longer R11.2, R6.1
- net N$36: now also 1F1.2A, 1TH1.1; no longer D2.A, D4.C, L1.2
- net N$4: now also 2R10.1; no longer R10.1
- net N$40: now also 2R7.2; no longer R7.2
- net N$42: now also 3R6.1; no longer R156.1
- net N$7: now also 4DD1C.I1, 4DD1D.O; no longer DD1C.I0, DD1C.I1, DD1D.O
Other:
- note removed: "5"
- note removed: "9"
- moved on the sheet: PCB_PW, PCB_SW

Commit message: .
Parts:
- removed OK1: PC817, optocoupler:PC817
- added 1PC1: PC817, optocoupler:PC817
- added 3CN1: (no value), 3do:FTOP-18
- added 3VD3: 12v, diode:ZENER-DIODEDO34-7
- added 4R6: 100, rcl:R-EU_M0805
- 1R1: device rcl:R-EU_0613/15 -> rcl:R-EU_0309/12
- 2C4, 2C5, 2C7: value (none) -> 330
- 2C6: device rcl:C-EUC1206 -> rcl:C-EUC0805
- 2R5: value (none) -> 10k; device rcl:R-EU_R1206 -> rcl:R-EU_M0805
- 2R7: value (none) -> 10k
- 2R8: value (none) -> 68k *80ruw
- 2R9: value (none) -> 100
- 2VD1: value 1N4148DO35-10 -> 1N4148
- 2VD2: value 1N4148DO35-7 -> FR207; device diode:1N4148DO35-7 -> diode:1N4148DO35-10
- 2VD3: value 1N4148DO35-7 -> LL4148; device diode:1N4148DO35-7 -> diode:DIODE-SOD80C
- 3C1: value (none) -> 560mfx25v
- 3C2: value 100mfx25v -> 1000mfx25v
- 3C5: value (none) -> 470vfx25v
- 4VD3: value 1N4148DO35-7 -> (none); device diode:1N4148DO35-7 -> diode:DIODE-SOD80C
Connections:
- removed net +9V: 3C5.+, 3L1.2, 3R5A.2, 3R7.2, J9V.1
- new net N$38: 3C5.+, 3CN1-1.1, 3CN1-2.1, 3CN1-3.1, 3L1.2, 3R5A.2, 3R7.2, 3VD3.C, J9V.1
- new net N$44: 1C2.1, 1L1.4, 1VD1B.AC1, 1VD2.A, 1VD4.C
- net +5V: now also 3CN1-13.1, 3CN1-14.1, 3CN1-15.1, 3CN1-16.1, 3CN1-17.1
- net GND: now also 2T1.9V2, 3CN1-10.1, 3CN1-11.1, 3CN1-12.1, 3CN1-4.1, 3CN1-5.1, 3CN1-6.1, 3CN1-7.1, 3CN1-8.1, 3CN1-9.1, 3VD3.A; no longer 2T1.O1.2
- net MON: now also 3CN1-18.1, 4R6.2; no longer 4R5.1, 4VT1.C
- net N$12: now also 1PC1.C; no longer OK1.C
- net N$13: now also 1PC1.A; no longer OK1.A
- net N$15: now also 1C2.2, 1L1.2; no longer 1C2.1, 1L1.4
- net N$20: now also 1PC1.COL; no longer OK1.COL
- net N$29: now also 4R5.1, 4R6.1, 4VT1.C; no longer 1C2.2, 1L1.2, 1VD1B.AC1, 1VD2.A, 1VD4.C
- net N$40: now also 1PC1.EMIT; no longer OK1.EMIT
- net N$5: now also 2T1.9V1; no longer 2T1.O1.1
Other:
- moved on the sheet: 1C1, 1C2, 1C7, 1DA1, 1F1, 1L1, 1R1, 1RZ1, 1TH1, 1VD1, 1VD1B, 1VD2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

Commit message: .
Parts:
- 1C1: device 3do:C26X19 -> 3do:C26X9
- 2R13: device rcl:R-EU_R1206 -> rcl:R-EU_0207/10
- 2R4, 2R9: device rcl:R-EU_R1206 -> rcl:R-EU_0204/7
- 2VD1: device diode:1N4148DO35-10 -> diode:1N4148DO35-7
- 2VD3: device diode:DIODE-SOD80C -> diode:1N4148DO35-7
- 2VD4: device diode:ZENER-DIODEDO34-7 -> diode:ZENER-DIODEDO35Z10
- 3R5C: device rcl:R-EU_M1206 -> rcl:R-EU_0207/10
- 4C2A: value (none) -> 3p
Connections:
- net N$15: now also 1C2.1, 1L1.4; no longer 1C2.2, 1L1.2
- net N$19: no longer 4R1B.2, 4R1C.A, 4VD2.A
- net N$44: now also 1C2.2, 1L1.2; no longer 1C2.1, 1L1.4
- net N$7: now also 4R1B.2, 4R1C.A, 4VD2.A
Other:
- moved on the sheet: 1C1, 1C2, 1F1, 1L1, 1PC1, 1R1, 1RZ1, 1TH1, 2C10, 2R12, 2R13, 2R14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

Commit message: .
Parts:
- removed 4C2B: (no value), rcl:C-EU050-025X075
- removed 4C2D: (no value), rcl:C-EUC1206
- added 3R6B: 0, rcl:R-EU_0204/7
- 3R6: device rcl:R-EU_M1206 -> rcl:R-EU_0204/7
- 4R6: device rcl:R-EU_M0805 -> rcl:R-EU_R1206
Connections:
- new net N$43: 3R6.1, 3R6B.2
- net N$1: now also 4DD1D.I0, 4DD1D.I1; no longer 4C2B.2, 4C2D.2, 4DD1A.I0, 4DD1A.I1
- net N$19: now also 4DD1A.I0, 4DD1A.I1, 4DD1C.O; no longer 4C2B.1, 4C2D.1, 4DD1B.O, 4DD1D.I0, 4DD1D.I1
- net N$2: now also 4DD1C.I0, 4DD1C.I1, 4DD1D.O; no longer 4DD1A.O, 4DD1B.I0, 4DD1B.I1
- net N$25: now also 4DD1B.O; no longer 4DD1C.O
- net N$31: now also 4DD1B.I1; no longer 4DD1C.I0
- net N$42: now also 3R6B.1; no longer 3R6.1
- net N$7: now also 4DD1A.O, 4DD1B.I0; no longer 4DD1C.I1, 4DD1D.O
Other:
- note added: "1"
- note added: "10"
- note added: "11"
- note added: "2"
- note added: "4"
- note added: "5"
- note added: "6"
- note added: "7"
- moved on the sheet: 3R6, 4C2C, 4DD1A, 4DD1B, 4DD1C, 4DD1D

Commit message: .
Parts:
- 2R8: value 68k *80ruw -> 68k *80khz
- 2VD4: value (none) -> 22v
- 4C1: value (none) -> 100n
Connections:
- net N$9 renamed +16IN
- removed net N$36: 1F1.2A, 1TH1.1
- new net N$9: 1TH1.1, PCB_SW.P
- net N$32: now also 1TH1.2; no longer PCB_SW.P
- net N$33: now also 1F1.2A; no longer 1TH1.2
Other:
- note added: "github.com/74ls00/3do"
- moved on the sheet: 1C1, 1C2, 1F1, 1L1, 1R1, 1RZ1, 1TH1, PCB_PW, PCB_SW

Commit message: .
Parts:
- removed 1VD1B: S1WBS60, rectifier:B-DIL
- removed 4R2: 4k7, rcl:R-EU_R1206
- added 4C3A: (no value), rcl:C-EUC1812
- 4R3: value 4k7 -> 270k
- 4VD3: value (none) -> LL4148
Connections:
- removed net N$31: 4DD1B.I1, 4R2.1, 4R3.2
- net +5V: now also 4R3.2, 4VD3.C; no longer 4C3.+
- net -IN: no longer 1VD1B.-
- net GND: now also 4C3.-, 4C3A.2; no longer 4R3.1, 4VD3.A
- net N$15: no longer 1VD1B.AC2
- net N$23: no longer 1VD1B.+
- net N$35: now also 4C3.+, 4C3A.1, 4DD1B.I1, 4R3.1, 4VD3.A; no longer 4C3.-, 4R2.2, 4VD3.C
- net N$44: no longer 1VD1B.AC1
Other:
- note added: "3"
- moved on the sheet: 4C1, 4C3, 4DD1P, 4R3, 4VD3

Commit message: .
Parts:
- removed 2R11A, 2R11B, 2R11C, 2R11D: 1, rcl:R-EU_R0805
- added 2R11: (no value), rcl:R-EU_0613/15
- 2VD1: device diode:1N4148DO35-7 -> diode:1N4148DO35-10
Connections:
- removed net N$21: 2R11A.2, 2R11B.2, 2VT1.S
- net -IN: now also 2R11.1; no longer 2R11C.1, 2R11D.1
- net N$37: now also 2R11.2, 2VT1.S; no longer 2R11A.1, 2R11B.1, 2R11C.2, 2R11D.2
Other:
- moved on the sheet: 1C1, 1C2, 1F1, 1L1, 1R1, 1RZ1, 1TH1, 1VD1, 1VD3, 2R10, 4C1, 4C2A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

Commit message: .
Parts:
- 2C11: device rcl:C-EU050-025X075 -> rcl:C-EU075-032X103
Changed lines of the file:
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@@
 <part name="2VD1" library="diode" deviceset="1N4148" device="DO35-10" value="1N4148"/>
 <part name="2R4" library="rcl" deviceset="R-EU_" device="0204/7" value="22"/>
-<part name="2C11" library="rcl" deviceset="C-EU" device="050-025X075" value="4n7"/>
+<part name="2C11" library="rcl" deviceset="C-EU" device="075-032X103" value="4n7"/>
 <part name="GND4" library="supply1" deviceset="GND" device=""/>
 <part name="1F1" library="fuse" deviceset="SHK20L" device=""/>
