File: fz10_pow.sch (EAGLE design)
At the start: 80 parts

Commit message: .
Parts:
- 2C2: device rcl:C-EU050-025X075 -> rcl:C-EU075-032X103
Changed lines of the file:
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@@
 <part name="2R10" library="rcl" deviceset="R-EU_" device="R1206" value="1k"/>
 <part name="2T1" library="3do" deviceset="TRANS_ER29" device=""/>
-<part name="2C2" library="rcl" deviceset="C-EU" device="050-025X075" value="10n"/>
+<part name="2C2" library="rcl" deviceset="C-EU" device="075-032X103" value="10n"/>
 <part name="2VD1" library="diode" deviceset="1N4148" device="DO35-10" value="1N4148"/>
 <part name="2R4" library="rcl" deviceset="R-EU_" device="0204/7" value="22"/>
@@
 <plain>
 <text x="162.56" y="93.98" size="1.778" layer="91" rot="R180">1</text>
-<text x="162.56" y="83.82" size="1.778" layer="91" rot="R180">2</text>
-<text x="162.56" y="101.6" size="1.778" layer="91" rot="R180">3</text>
+<text x="162.56" y="101.6" size="1.778" layer="91" rot="R180">2</text>
+<text x="162.56" y="83.82" size="1.778" layer="91" rot="R180">3</text>
 <text x="162.56" y="111.76" size="1.778" layer="91" rot="R180">5</text>
 <text x="180.34" y="101.6" size="1.778" layer="91" rot="R180">6</text>

Commit message: .
Parts:
- 2VD1: device diode:1N4148DO35-10 -> diode:DIODE-SOD80C
Other:
- note removed: "1"
- note removed: "10"
- note removed: "11"
- note removed: "2"
- note removed: "3"
- note removed: "4"
- note removed: "5"
- note removed: "6"
- note removed: "7"
Changed lines of the file:
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@@
 <part name="2T1" library="3do" deviceset="TRANS_ER29" device=""/>
 <part name="2C2" library="rcl" deviceset="C-EU" device="075-032X103" value="10n"/>
-<part name="2VD1" library="diode" deviceset="1N4148" device="DO35-10" value="1N4148"/>
+<part name="2VD1" library="diode" deviceset="DIODE-" device="SOD80C" value="1N4148"/>
 <part name="2R4" library="rcl" deviceset="R-EU_" device="0204/7" value="22"/>
 <part name="2C11" library="rcl" deviceset="C-EU" device="075-032X103" value="4n7"/>
@@
 <sheet>
 <plain>
-<text x="162.56" y="93.98" size="1.778" layer="91" rot="R180">1</text>
-<text x="162.56" y="101.6" size="1.778" layer="91" rot="R180">2</text>
-<text x="162.56" y="83.82" size="1.778" layer="91" rot="R180">3</text>
-<text x="162.56" y="111.76" size="1.778" layer="91" rot="R180">5</text>
-<text x="180.34" y="101.6" size="1.778" layer="91" rot="R180">6</text>
-<text x="180.34" y="111.76" size="1.778" layer="91" rot="R180">7</text>
-<text x="180.34" y="83.82" size="1.778" layer="91" rot="R180">10</text>
-<text x="180.34" y="93.98" size="1.778" layer="91" rot="R180">11</text>
 <text x="33.02" y="157.48" size="3.81" layer="91">github.com/74ls00/3do</text>
-<text x="162.56" y="106.68" size="1.778" layer="91" rot="R180">4</text>
 </plain>
 <instances>

Commit message: .
Parts:
- 2R10: value 1k -> 470
- 2R11: value (none) -> 1
- 2VD1: value 1N4148 -> LL4148
Changed lines of the file:
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@@
 <grid distance="100" unitdist="mil" unit="mil" style="lines" multiple="1" display="yes" altdistance="0.01" altunitdist="inch" altunit="inch"/>
 <layers>
-<layer number="1" name="Top" color="4" fill="1" visible="yes" active="no"/>
-<layer number="2" name="Route2" color="1" fill="3" visible="yes" active="no"/>
-<layer number="3" name="Route3" color="4" fill="3" visible="yes" active="no"/>
-<layer number="4" name="Route4" color="1" fill="4" visible="yes" active="no"/>
-<layer number="5" name="Route5" color="4" fill="4" visible="yes" active="no"/>
-<layer number="6" name="Route6" color="1" fill="8" visible="yes" active="no"/>
-<layer number="7" name="Route7" color="4" fill="8" visible="yes" active="no"/>
-<layer number="8" name="Route8" color="1" fill="2" visible="yes" active="no"/>
-<layer number="9" name="Route9" color="4" fill="2" visible="yes" active="no"/>
-<layer number="10" name="Route10" color="1" fill="7" visible="yes" active="no"/>
-<layer number="11" name="Route11" color="4" fill="7" visible="yes" active="no"/>
-<layer number="12" name="Route12" color="1" fill="5" visible="yes" active="no"/>
-<layer number="13" name="Route13" color="4" fill="5" visible="yes" active="no"/>
-<layer number="14" name="Route14" color="1" fill="6" visible="yes" active="no"/>
-<layer number="15" name="Route15" color="4" fill="6" visible="yes" active="no"/>
-<layer number="16" name="Bottom" color="1" fill="1" visible="yes" active="no"/>
-<layer number="17" name="Pads" color="2" fill="1" visible="yes" active="no"/>
-<layer number="18" name="Vias" color="2" fill="1" visible="yes" active="no"/>
-<layer number="19" name="Unrouted" color="6" fill="1" visible="yes" active="no"/>
-<layer number="20" name="Dimension" color="15" fill="1" visible="yes" active="no"/>
-<layer number="21" name="tPlace" color="7" fill="1" visible="yes" active="no"/>
-<layer number="22" name="bPlace" color="7" fill="1" visible="yes" active="no"/>
-<layer number="23" name="tOrigins" color="15" fill="1" visible="yes" active="no"/>
-<layer number="24" name="bOrigins" color="15" fill="1" visible="yes" active="no"/>
-<layer number="25" name="tNames" color="7" fill="1" visible="yes" active="no"/>
-<layer number="26" name="bNames" color="7" fill="1" visible="yes" active="no"/>
-<layer number="27" name="tValues" color="7" fill="1" visible="yes" active="no"/>
-<layer number="28" name="bValues" color="7" fill="1" visible="yes" active="no"/>
+<layer number="1" name="Top" color="4" fill="1" visible="no" active="no"/>
+<layer number="2" name="Route2" color="1" fill="3" visible="no" active="no"/>
+<layer number="3" name="Route3" color="4" fill="3" visible="no" active="no"/>
+<layer number="4" name="Route4" color="1" fill="4" visible="no" active="no"/>
+<layer number="5" name="Route5" color="4" fill="4" visible="no" active="no"/>
+<layer number="6" name="Route6" color="1" fill="8" visible="no" active="no"/>
+<layer number="7" name="Route7" color="4" fill="8" visible="no" active="no"/>
+<layer number="8" name="Route8" color="1" fill="2" visible="no" active="no"/>
+<layer number="9" name="Route9" color="4" fill="2" visible="no" active="no"/>
+<layer number="10" name="Route10" color="1" fill="7" visible="no" active="no"/>
+<layer number="11" name="Route11" color="4" fill="7" visible="no" active="no"/>
+<layer number="12" name="Route12" color="1" fill="5" visible="no" active="no"/>
+<layer number="13" name="Route13" color="4" fill="5" visible="no" active="no"/>
+<layer number="14" name="Route14" color="1" fill="6" visible="no" active="no"/>
+<layer number="15" name="Route15" color="4" fill="6" visible="no" active="no"/>
+<layer number="16" name="Bottom" color="1" fill="1" visible="no" active="no"/>
+<layer number="17" name="Pads" color="2" fill="1" visible="no" active="no"/>
+<layer number="18" name="Vias" color="2" fill="1" visible="no" active="no"/>
+<layer number="19" name="Unrouted" color="6" fill="1" visible="no" active="no"/>
+<layer number="20" name="Dimension" color="15" fill="1" visible="no" active="no"/>
+<layer number="21" name="tPlace" color="7" fill="1" visible="no" active="no"/>
+<layer number="22" name="bPlace" color="7" fill="1" visible="no" active="no"/>
+<layer number="23" name="tOrigins" color="15" fill="1" visible="no" active="no"/>
+<layer number="24" name="bOrigins" color="15" fill="1" visible="no" active="no"/>
+<layer number="25" name="tNames" color="7" fill="1" visible="no" active="no"/>
+<layer number="26" name="bNames" color="7" fill="1" visible="no" active="no"/>
+<layer number="27" name="tValues" color="7" fill="1" visible="no" active="no"/>
+<layer number="28" name="bValues" color="7" fill="1" visible="no" active="no"/>
 <layer number="29" name="tStop" color="7" fill="3" visible="no" active="no"/>
 <layer number="30" name="bStop" color="7" fill="6" visible="no" active="no"/>
@@
 <layer number="35" name="tGlue" color="7" fill="4" visible="no" active="no"/>
 <layer number="36" name="bGlue" color="7" fill="5" visible="no" active="no"/>
-<layer number="37" name="tTest" color="7" fill="1" visible="yes" active="no"/>
-<layer number="38" name="bTest" color="7" fill="1" visible="yes" active="no"/>
+<layer number="37" name="tTest" color="7" fill="1" visible="no" active="no"/>
+<layer number="38" name="bTest" color="7" fill="1" visible="no" active="no"/>
 <layer number="39" name="tKeepout" color="4" fill="11" visible="no" active="no"/>
 <layer number="40" name="bKeepout" color="1" fill="11" visible="no" active="no"/>
@@
 <layer number="44" name="Drills" color="7" fill="1" visible="no" active="no"/>
 <layer number="45" name="Holes" color="7" fill="1" visible="no" active="no"/>
-<layer number="46" name="Milling" color="3" fill="1" visible="yes" active="no"/>
-<layer number="47" name="Measures" color="7" fill="1" visible="yes" active="no"/>
-<layer number="48" name="Document" color="7" fill="1" visible="yes" active="no"/>
-<layer number="49" name="Reference" color="7" fill="1" visible="yes" active="no"/>
-<layer number="50" name="dxf" color="7" fill="1" visible="yes" active="no"/>
-<layer number="51" name="tDocu" color="7" fill="1" visible="yes" active="no"/>
-<layer number="52" name="bDocu" color="7" fill="1" visible="yes" active="no"/>
-<layer number="53" name="tGND_GNDA" color="7" fill="1" visible="yes" active="no"/>
-<layer number="54" name="bGND_GNDA" color="7" fill="1" visible="yes" active="no"/>
-<layer number="56" name="wert" color="7" fill="1" visible="yes" active="no"/>
-<layer number="57" name="tCAD" color="7" fill="1" visible="yes" active="no"/>
+<layer number="46" name="Milling" color="3" fill="1" visible="no" active="no"/>
+<layer number="47" name="Measures" color="7" fill="1" visible="no" active="no"/>
+<layer number="48" name="Document" color="7" fill="1" visible="no" active="no"/>
+<layer number="49" name="Reference" color="7" fill="1" visible="no" active="no"/>
+<layer number="50" name="dxf" color="7" fill="1" visible="no" active="no"/>
+<layer number="51" name="tDocu" color="7" fill="1" visible="no" active="no"/>
+<layer number="52" name="bDocu" color="7" fill="1" visible="no" active="no"/>
+<layer number="53" name="tGND_GNDA" color="7" fill="1" visible="no" active="no"/>
+<layer number="54" name="bGND_GNDA" color="7" fill="1" visible="no" active="no"/>
+<layer number="56" name="wert" color="7" fill="1" visible="no" active="no"/>
+<layer number="57" name="tCAD" color="7" fill="1" visible="no" active="no"/>
 <layer number="90" name="Modules" color="7" fill="1" visible="yes" active="yes"/>
 <layer number="91" name="Nets" color="2" fill="1" visible="yes" active="yes"/>
@@
 <part name="1C7" library="rcl" deviceset="CPOL-EU" device="E10-22.5" value="47x400v"/>
 <part name="2VT1" library="transistor-power" deviceset="IRF3704" device="L-V"/>
-<part name="2R10" library="rcl" deviceset="R-EU_" device="R1206" value="1k"/>
+<part name="2R10" library="rcl" deviceset="R-EU_" device="R1206" value="470"/>
 <part name="2T1" library="3do" deviceset="TRANS_ER29" device=""/>
 <part name="2C2" library="rcl" deviceset="C-EU" device="075-032X103" value="10n"/>
-<part name="2VD1" library="diode" deviceset="DIODE-" device="SOD80C" value="1N4148"/>
+<part name="2VD1" library="diode" deviceset="DIODE-" device="SOD80C" value="LL4148"/>
 <part name="2R4" library="rcl" deviceset="R-EU_" device="0204/7" value="22"/>
 <part name="2C11" library="rcl" deviceset="C-EU" device="075-032X103" value="4n7"/>
@@
 <part name="4C3A" library="rcl" deviceset="C-EU" device="C1812"/>
 <part name="GND14" library="supply1" deviceset="GND" device=""/>
-<part name="2R11" library="rcl" deviceset="R-EU_" device="0613/15"/>
+<part name="2R11" library="rcl" deviceset="R-EU_" device="0613/15" value="1"/>
 </parts>
 <sheets>
@@
 </instance>
 <instance part="2C3" gate="G$1" x="109.22" y="22.86" smashed="yes">
-<attribute name="NAME" x="105.283" y="30.9626" size="1.778" layer="95"/>
-<attribute name="VALUE" x="105.283" y="28.4226" size="1.778" layer="96"/>
+<attribute name="NAME" x="105.283" y="38.5826" size="1.778" layer="95"/>
+<attribute name="VALUE" x="105.283" y="36.0426" size="1.778" layer="96"/>
 </instance>
 <instance part="2R9" gate="G$1" x="119.38" y="81.28" smashed="yes">

Commit message: .
Parts:
- added 2R4B: (no value), rcl:R-EU_0207/10
- 2C11: value 4n7 -> 4n7 1kv
- 2R10: device rcl:R-EU_R1206 -> rcl:R-EU_0207/10
- 2R11: value 1 -> 0.91e
- 2R4: device rcl:R-EU_0204/7 -> rcl:R-EU_M0805
- 2R7: device rcl:R-EU_R1206 -> rcl:R-EU_R0805
- 2R8: value 68k *80khz -> 68k *(80khz); device rcl:R-EU_R1206 -> rcl:R-EU_R0805
- 2VD4: value 22v -> 22v(1n4748a)
- 3R5A: value 82k -> 30k
- 3R5B: value (none) -> 56k
- 3R5C: value (none) -> 560
- 3R6B: value 0 -> 0jp
- 3VD3: value 12v -> 12v(1n4742a)
- 4C1: device rcl:C-EUC1206 -> rcl:C-EUC0805
Connections:
- removed net N$37: 2R11.2, 2VT1.S
- new net N$21: 2R10.2, 2R11.2, 2VT1.S
- net +16IN: now also 2R4B.1
- net -IN: no longer 2R10.2
- net N$22: now also 2R4B.2
Other:
- note added: "2T1 ETD 29/16/10 2mm I 2-4 60w 2x0.2x0.2mm III 4-5 20w 2x0.2mm II 1-3 12w 0.2mm IV 6-7 4w 6x0.4mm V 10-11 7w 4x0.4mm"
- note added: "for FZ-10 REV 1.1"
- moved on the sheet: 1C7, 1DA1, 1VD1, 1VD2, 1VD3, 1VD4, 2C11, 2C2, 2C3, 2C4, 2C5, 2C6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

Commit message: .
Parts:
- 3VD3: value 12v(1n4742a) -> 12v(1N4742A)
- 4DD1: value 4011D -> CD4011BM
- 4R1C: value (none) -> 200k
Other:
- note added: "2T1 ETD 29/16/10 2mm I 2-4 62w 0.6mm III 4-5 20w 2x0.2mm II 1-3 12w 0.2mm IV 6-7 4w 6x0.6mm V 10-11 7w 4x0.6mm"
- note removed: "2T1 ETD 29/16/10 2mm I 2-4 60w 2x0.2x0.2mm III 4-5 20w 2x0.2mm II 1-3 12w 0.2mm IV 6-7 4w 6x0.4mm V 10-11 7w 4x0.4mm"
- moved on the sheet: 3CN1-1, 3CN1-10, 3CN1-11, 3CN1-12, 3CN1-18, 3CN1-2, 3CN1-3, 3CN1-4, 3CN1-5, 3CN1-6, 3CN1-7, 3CN1-8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

Commit message: .
Parts:
- removed 4C3A: (no value), rcl:C-EUC1812
- added 4C3B: (no value), rcl:CPOL-EUE2.5-5
- 2VT1: value IRF3704L-V -> 2SK1984
- 3VD1: value BYV32 -> FCB06A06
- 3VD2: value BYV32 -> MA10799
- 4C3: value 4m7 -> 10m; device rcl:CPOL-EUE2.5-5 -> rcl:C-EUC1812
Connections:
- net GND: now also 4C3.2, 4C3B.-; no longer 4C3.-, 4C3A.2
- net N$35: now also 4C3.1, 4C3B.+; no longer 4C3.+, 4C3A.1
Other:
- note added: "2T1 ETD 29/16/10 2mm I 2-4 62w 0.6mm III 4-5 20w 0.6mm II 1-3 12w 0.2mm IV 6-7 4w 6x0.6mm V 10-11 7w 4x0.6mm"
- note added: "3L1 ~2mkHn 3X10mm 13w 0.5mm"
- note added: "3L1 ~5mkHn 6X12mm 15w 0.5mm"
- note removed: "2T1 ETD 29/16/10 2mm I 2-4 62w 0.6mm III 4-5 20w 2x0.2mm II 1-3 12w 0.2mm IV 6-7 4w 6x0.6mm V 10-11 7w 4x0.6mm"
- moved on the sheet: 1C7, 1VD1, 1VD2, 1VD3, 1VD4, 2C10, 2C4, 2C5, 2C7, 2R10, 2R11, 2R12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

Commit message: .
Parts:
- renumbered 4C2C to 4C2B, 4C3 to 4C3A
Other:
- moved on the sheet: PCB_SW
Changed lines of the file:
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@@
 <part name="4VD2" library="diode" deviceset="DIODE-" device="SOD80C" value="LL4158"/>
 <part name="4C1" library="rcl" deviceset="C-EU" device="C0805" value="100n"/>
-<part name="4C2C" library="rcl" deviceset="C-EU" device="C1206"/>
+<part name="4C2B" library="rcl" deviceset="C-EU" device="C1206"/>
 <part name="1DA1" library="v-reg" deviceset="UC384*" device="N" technology="2"/>
 <part name="1PC1" library="optocoupler" deviceset="PC817" device=""/>
@@
 <part name="GND13" library="supply1" deviceset="GND" device=""/>
 <part name="P+1" library="supply1" deviceset="+5V" device=""/>
-<part name="4C3" library="rcl" deviceset="C-EU" device="C1812" value="10m"/>
+<part name="4C3A" library="rcl" deviceset="C-EU" device="C1812" value="10m"/>
 <part name="GND14" library="supply1" deviceset="GND" device=""/>
 <part name="2R11" library="rcl" deviceset="R-EU_" device="0613/15" value="0.91e"/>
@@
 </plain>
 <instances>
-<instance part="PCB" gate="_SW" x="96.52" y="124.46" smashed="yes" rot="MR180">
-<attribute name="NAME" x="92.075" y="119.38" size="1.778" layer="95" rot="MR180"/>
-<attribute name="VALUE" x="89.535" y="116.84" size="1.778" layer="96" rot="MR180"/>
+<instance part="PCB" gate="_SW" x="96.52" y="124.46" smashed="yes">
+<attribute name="NAME" x="92.075" y="121.92" size="1.778" layer="95"/>
+<attribute name="VALUE" x="89.535" y="119.38" size="1.778" layer="96"/>
 </instance>
 <instance part="4DD1" gate="D" x="127" y="144.78" smashed="yes">
@@
 </instance>
 <instance part="4VD1" gate="G$1" x="132.08" y="167.64" smashed="yes">
-<attribute name="NAME" x="127" y="173.2026" size="1.778" layer="95"/>
-<attribute name="VALUE" x="142.24" y="175.0314" size="1.778" layer="96" rot="R180"/>
+<attribute name="NAME" x="124.46" y="170.6626" size="1.778" layer="95"/>
+<attribute name="VALUE" x="142.24" y="172.4914" size="1.778" layer="96" rot="R180"/>
 </instance>
 <instance part="4VD2" gate="G$1" x="162.56" y="167.64" smashed="yes" rot="R180">
-<attribute name="NAME" x="152.4" y="173.2026" size="1.778" layer="95"/>
-<attribute name="VALUE" x="170.18" y="175.0314" size="1.778" layer="96" rot="R180"/>
+<attribute name="NAME" x="152.4" y="170.6626" size="1.778" layer="95"/>
+<attribute name="VALUE" x="170.18" y="172.4914" size="1.778" layer="96" rot="R180"/>
 </instance>
 <instance part="4DD1" gate="P" x="185.42" y="154.94" smashed="yes">
@@
 <attribute name="VALUE" x="192.024" y="157.861" size="1.778" layer="96"/>
 </instance>
-<instance part="4C2C" gate="G$1" x="137.16" y="127" smashed="yes" rot="R270">
-<attribute name="NAME" x="123.444" y="127.381" size="1.778" layer="95"/>
+<instance part="4C2B" gate="G$1" x="137.16" y="127" smashed="yes" rot="R270">
+<attribute name="NAME" x="125.984" y="127.381" size="1.778" layer="95"/>
 <attribute name="VALUE" x="132.461" y="125.476" size="1.778" layer="96" rot="R270"/>
 </instance>
@@
 <attribute name="VALUE" x="193.04" y="172.72" size="1.778" layer="96" rot="R180"/>
 </instance>
-<instance part="4C3" gate="G$1" x="198.12" y="144.78" smashed="yes" rot="MR0">
-<attribute name="NAME" x="192.024" y="146.939" size="1.778" layer="95" rot="MR180"/>
-<attribute name="VALUE" x="196.596" y="140.081" size="1.778" layer="96" rot="MR0"/>
+<instance part="4C3A" gate="G$1" x="198.12" y="144.78" smashed="yes" rot="MR0">
+<attribute name="NAME" x="188.976" y="140.081" size="1.778" layer="95" rot="MR0"/>
+<attribute name="VALUE" x="188.976" y="137.541" size="1.778" layer="96" rot="MR0"/>
 </instance>
 <instance part="GND14" gate="1" x="198.12" y="134.62"/>
@@
 <junction x="116.84" y="142.24"/>
 <wire x1="116.84" y1="134.62" x2="116.84" y2="127" width="0.1524" layer="91"/>
-<pinref part="4C2C" gate="G$1" pin="2"/>
+<pinref part="4C2B" gate="G$1" pin="2"/>
 <wire x1="116.84" y1="127" x2="132.08" y2="127" width="0.1524" layer="91"/>
 <junction x="116.84" y="134.62"/>
@@
 <segment>
 <pinref part="GND14" gate="1" pin="GND"/>
-<pinref part="4C3" gate="G$1" pin="2"/>
+<pinref part="4C3A" gate="G$1" pin="2"/>
 <wire x1="198.12" y1="137.16" x2="198.12" y2="139.7" width="0.1524" layer="91"/>
 </segment>
@@
 <wire x1="157.48" y1="134.62" x2="157.48" y2="139.7" width="0.1524" layer="91"/>
 <wire x1="157.48" y1="139.7" x2="157.48" y2="144.78" width="0.1524" layer="91"/>
-<pinref part="4C2C" gate="G$1" pin="1"/>
+<pinref part="4C2B" gate="G$1" pin="1"/>
 <wire x1="139.7" y1="127" x2="157.48" y2="127" width="0.1524" layer="91"/>
 <wire x1="157.48" y1="127" x2="157.48" y2="134.62" width="0.1524" layer="91"/>
@@
 <wire x1="210.82" y1="154.94" x2="210.82" y2="149.86" width="0.1524" layer="91"/>
 <junction x="210.82" y="149.86"/>
-<pinref part="4C3" gate="G$1" pin="1"/>
+<pinref part="4C3A" gate="G$1" pin="1"/>
 <wire x1="198.12" y1="147.32" x2="198.12" y2="149.86" width="0.1524" layer="91"/>
 <wire x1="198.12" y1="149.86" x2="205.74" y2="149.86" width="0.1524" layer="91"/>

Commit message: .
Parts:
- added 2C12: 100n, rcl:C-EUC0805
- 2R16: value 3k3 -> 10k
- 4VD2: value LL4158 -> LL4148
Connections:
- net +16IN: now also 2C12.1
- net -IN: now also 2C12.2
Other:
- note added: "2T1 ETD 29/16/10 2mm I 2-4 62w 0.6mm II 4-5 20w 0.6mm III 1-3 12w 0.2mm IV 6-7 4w 6x0.6mm V 10-11 7w 4x0.6mm"
- note removed: "2T1 ETD 29/16/10 2mm I 2-4 62w 0.6mm III 4-5 20w 0.6mm II 1-3 12w 0.2mm IV 6-7 4w 6x0.6mm V 10-11 7w 4x0.6mm"
- moved on the sheet: 2C6, 2R16, 3C3, 3R6B
