File: fz10_pow.sch (EAGLE design)
At the start: 82 parts

Commit message: .
Parts:
- 2R16: value 10k -> 8k2
- 3R5A: value 30k -> (none)
- 3R5B: value 56k -> (none)
- 3R5C: value 560 -> (none)
- 3R6: value 3k9 -> 9k1
- 3R7: value 100 -> 82
Other:
- note added: "2T1 ETD 29/16/10 2mm I 2-4 51w 0.4mm II 4-5 51w 0.4mm III 1-3 17w 0.2mm IV 6-7 5w 6x0.55mm V 10-11 8w 4x0.55mm"
- note removed: "2T1 ETD 29/16/10 2mm I 2-4 62w 0.6mm II 4-5 20w 0.6mm III 1-3 12w 0.2mm IV 6-7 4w 6x0.6mm V 10-11 7w 4x0.6mm"
Changed lines of the file:
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@@
 <part name="2R14" library="rcl" deviceset="R-EU_" device="R1206" value="47k*"/>
 <part name="2C10" library="rcl" deviceset="C-EU" device="050-025X075" value="10n*"/>
-<part name="2R16" library="rcl" deviceset="R-EU_" device="R1206" value="10k"/>
+<part name="2R16" library="rcl" deviceset="R-EU_" device="R1206" value="8k2"/>
 <part name="GND2" library="supply1" deviceset="GND" device=""/>
 <part name="GND3" library="supply1" deviceset="GND" device=""/>
@@
 <part name="3C5" library="rcl" deviceset="CPOL-EU" device="E5-8.5" value="470vfx25v"/>
 <part name="GND11" library="supply1" deviceset="GND" device=""/>
-<part name="3R7" library="rcl" deviceset="R-EU_" device="0613/15" value="100"/>
+<part name="3R7" library="rcl" deviceset="R-EU_" device="0613/15" value="82"/>
 <part name="GND12" library="supply1" deviceset="GND" device=""/>
-<part name="3R5A" library="rcl" deviceset="R-EU_" device="M1206" value="30k"/>
-<part name="3R5B" library="rcl" deviceset="R-EU_" device="M1206" value="56k"/>
-<part name="3R5C" library="rcl" deviceset="R-EU_" device="0207/10" value="560"/>
-<part name="3R6" library="rcl" deviceset="R-EU_" device="0204/7" value="3k9"/>
+<part name="3R5A" library="rcl" deviceset="R-EU_" device="M1206"/>
+<part name="3R5B" library="rcl" deviceset="R-EU_" device="M1206"/>
+<part name="3R5C" library="rcl" deviceset="R-EU_" device="0207/10"/>
+<part name="3R6" library="rcl" deviceset="R-EU_" device="0204/7" value="9k1"/>
 <part name="1C2" library="rcl" deviceset="C-EU" device="150-084X183" value="100nX250v"/>
 <part name="1RZ1" library="varistor" deviceset="S1210" device="" value=""/>
@@
 <text x="33.02" y="149.86" size="3.81" layer="91">for FZ-10 REV 1.1</text>
 <text x="45.72" y="106.68" size="1.778" layer="91" font="vector" rot="MR180">2T1 ETD 29/16/10 2mm
-I   2-4 62w 0.6mm
-II 4-5 20w 0.6mm
-III  1-3 12w 0.2mm
-IV 6-7 4w 6x0.6mm
-V 10-11 7w 4x0.6mm</text>
+I   2-4 51w 0.4mm
+II 4-5 51w 0.4mm
+III  1-3 17w 0.2mm
+IV 6-7 5w 6x0.55mm
+V 10-11 8w 4x0.55mm</text>
 <text x="276.86" y="127" size="1.778" layer="91" rot="MR180">3L1 ~2mkHn
 3X10mm

Commit message: .
Parts:
- added 2VD5: 1N4148, diode:1N4148DO35-7
- 2R16: value 8k2 -> 8.20k
- 2VD3: value LL4148 -> 1N4148
- 3R6: value 9k1 -> 8.32k
Connections:
- new net N$45: 2VD5.A
- net N$5: now also 2VD5.C
Other:
- moved on the sheet: 3CN1-18, 4C1, 4C2A, 4C2B, 4C3A, 4C3B, 4DD1A, 4DD1B, 4DD1C, 4DD1D, 4DD1P, 4R1A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
